File: Cleanroom Nano.sch (EAGLE design)
At the start: 23 parts, among them J001 USB_MICROB_JST, J002 M15, J003 M15, U001 FT232RLSSOP, U401 ATMEGA168, Y401 16MHz

Commit message: FT232 close to USB port, ATMega still diagonal
Connections:
- net N$10 renamed RXLED1
- net N$7 renamed TXLED1
- removed net RXC/D0: J002.2, U001.TXD, U401.PD0(RXD)
- removed net TXC/D1: J002.1, U001.RXD, U401.PD1(TXD)
- new net D0: J002.1, U001.TXD, U401.PD0(RXD)
- new net D1: J002.2, U001.RXD, U401.PD1(TXD)
Other:
- moved on the sheet: C002, D402, R001A
Changed lines of the file:
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@@
 <instance part="P+1" gate="1" x="-10.16" y="99.06"/>
 <instance part="GND1" gate="1" x="-2.54" y="7.62"/>
-<instance part="C002" gate="G$1" x="99.06" y="68.58" rot="R90"/>
+<instance part="C002" gate="G$1" x="104.14" y="73.66" rot="R90"/>
 <instance part="C017" gate="G$1" x="147.32" y="66.04"/>
 <instance part="P+2" gate="1" x="149.86" y="96.52"/>
@@
 <instance part="R001" gate="B" x="106.68" y="45.72" rot="R90"/>
 <instance part="R001" gate="C" x="96.52" y="45.72" rot="R90"/>
-<instance part="R001" gate="A" x="81.28" y="43.18" rot="R90"/>
+<instance part="R001" gate="A" x="86.36" y="45.72" rot="R90"/>
 <instance part="D401" gate="G$1" x="-22.86" y="45.72"/>
 <instance part="D001" gate="G$1" x="96.52" y="33.02"/>
 <instance part="D002" gate="G$1" x="106.68" y="33.02"/>
-<instance part="D402" gate="G$1" x="81.28" y="33.02"/>
+<instance part="D402" gate="G$1" x="86.36" y="33.02"/>
 <instance part="P+3" gate="1" x="127" y="33.02"/>
 <instance part="C004" gate="G$1" x="170.18" y="53.34"/>
@@
 <wire x1="-22.86" y1="40.64" x2="-22.86" y2="15.24" width="0.1524" layer="91"/>
 <wire x1="-22.86" y1="15.24" x2="-12.7" y2="15.24" width="0.1524" layer="91"/>
-<wire x1="81.28" y1="27.94" x2="81.28" y2="15.24" width="0.1524" layer="91"/>
+<wire x1="86.36" y1="27.94" x2="86.36" y2="15.24" width="0.1524" layer="91"/>
 <wire x1="142.24" y1="58.42" x2="147.32" y2="58.42" width="0.1524" layer="91"/>
 <wire x1="147.32" y1="63.5" x2="147.32" y2="60.96" width="0.1524" layer="91"/>
@@
 <wire x1="142.24" y1="50.8" x2="147.32" y2="50.8" width="0.1524" layer="91"/>
 <wire x1="147.32" y1="50.8" x2="147.32" y2="15.24" width="0.1524" layer="91"/>
-<wire x1="147.32" y1="15.24" x2="81.28" y2="15.24" width="0.1524" layer="91"/>
+<wire x1="147.32" y1="15.24" x2="86.36" y2="15.24" width="0.1524" layer="91"/>
 <wire x1="170.18" y1="15.24" x2="147.32" y2="15.24" width="0.1524" layer="91"/>
 <wire x1="170.18" y1="50.8" x2="170.18" y2="15.24" width="0.1524" layer="91"/>
@@
 <wire x1="180.34" y1="91.44" x2="177.8" y2="91.44" width="0.1524" layer="91"/>
 <wire x1="177.8" y1="91.44" x2="177.8" y2="15.24" width="0.1524" layer="91"/>
-<wire x1="5.08" y1="15.24" x2="81.28" y2="15.24" width="0.1524" layer="91"/>
+<wire x1="5.08" y1="15.24" x2="86.36" y2="15.24" width="0.1524" layer="91"/>
 <junction x="5.08" y="40.64"/>
 <junction x="5.08" y="38.1"/>
@@
 <junction x="170.18" y="15.24"/>
 <junction x="5.08" y="15.24"/>
-<junction x="81.28" y="15.24"/>
+<junction x="86.36" y="15.24"/>
 <pinref part="GND1" gate="1" pin="GND"/>
 <pinref part="U401" gate="G$1" pin="AGND"/>
@@
 </segment>
 </net>
-<net name="RXC/D0" class="0">
-<segment>
-<wire x1="68.58" y1="71.12" x2="76.2" y2="71.12" width="0.1524" layer="91"/>
-<wire x1="76.2" y1="71.12" x2="76.2" y2="83.82" width="0.1524" layer="91"/>
-<wire x1="76.2" y1="83.82" x2="83.82" y2="83.82" width="0.1524" layer="91"/>
-<label x="68.58" y="71.12" size="1.778" layer="95"/>
-<pinref part="U401" gate="G$1" pin="PD0(RXD)"/>
-<wire x1="96.52" y1="83.82" x2="96.52" y2="86.36" width="0.1524" layer="91"/>
-<wire x1="96.52" y1="86.36" x2="111.76" y2="86.36" width="0.1524" layer="91"/>
-<wire x1="93.98" y1="83.82" x2="96.52" y2="83.82" width="0.1524" layer="91"/>
-<pinref part="U001" gate="G$1" pin="TXD"/>
-<wire x1="83.82" y1="83.82" x2="93.98" y2="83.82" width="0" layer="91"/>
-</segment>
-<segment>
-<wire x1="-63.5" y1="96.52" x2="-73.66" y2="96.52" width="0.1524" layer="91"/>
-<label x="-73.66" y="96.52" size="1.778" layer="95"/>
-<pinref part="J002" gate="G$1" pin="2"/>
-</segment>
-</net>
-<net name="TXC/D1" class="0">
-<segment>
-<wire x1="68.58" y1="68.58" x2="78.74" y2="68.58" width="0.1524" layer="91"/>
-<wire x1="78.74" y1="68.58" x2="78.74" y2="76.2" width="0.1524" layer="91"/>
-<wire x1="78.74" y1="76.2" x2="83.82" y2="76.2" width="0.1524" layer="91"/>
-<label x="68.58" y="68.58" size="1.778" layer="95"/>
-<pinref part="U401" gate="G$1" pin="PD1(TXD)"/>
-<wire x1="101.6" y1="76.2" x2="101.6" y2="83.82" width="0.1524" layer="91"/>
-<wire x1="101.6" y1="83.82" x2="111.76" y2="83.82" width="0.1524" layer="91"/>
-<wire x1="93.98" y1="76.2" x2="101.6" y2="76.2" width="0.1524" layer="91"/>
-<pinref part="U001" gate="G$1" pin="RXD"/>
-<wire x1="83.82" y1="76.2" x2="93.98" y2="76.2" width="0" layer="91"/>
-</segment>
-<segment>
-<wire x1="-63.5" y1="99.06" x2="-73.66" y2="99.06" width="0.1524" layer="91"/>
-<label x="-73.66" y="99.06" size="1.778" layer="95"/>
-<pinref part="J002" gate="G$1" pin="1"/>
-</segment>
-</net>
 <net name="DTR#" class="0">
 <segment>
-<wire x1="106.68" y1="68.58" x2="106.68" y2="73.66" width="0.1524" layer="91"/>
-<wire x1="106.68" y1="73.66" x2="111.76" y2="73.66" width="0.1524" layer="91"/>
-<wire x1="106.68" y1="68.58" x2="101.6" y2="68.58" width="0.1524" layer="91"/>
+<wire x1="111.76" y1="73.66" x2="106.68" y2="73.66" width="0.1524" layer="91"/>
 <pinref part="U001" gate="G$1" pin="DTR"/>
 <pinref part="C002" gate="G$1" pin="2"/>
@@
 <net name="RESET" class="0">
 <segment>
-<wire x1="93.98" y1="68.58" x2="83.82" y2="68.58" width="0.1524" layer="91"/>
-<label x="83.82" y="68.58" size="1.778" layer="95"/>
+<wire x1="99.06" y1="73.66" x2="91.44" y2="73.66" width="0.1524" layer="91"/>
+<label x="91.44" y="73.66" size="1.778" layer="95"/>
 <pinref part="C002" gate="G$1" pin="1"/>
 </segment>
@@
 <net name="D13" class="0">
 <segment>
-<wire x1="68.58" y1="35.56" x2="73.66" y2="35.56" width="0.1524" layer="91"/>
-<wire x1="73.66" y1="35.56" x2="73.66" y2="53.34" width="0.1524" layer="91"/>
-<wire x1="73.66" y1="53.34" x2="81.28" y2="53.34" width="0.1524" layer="91"/>
-<wire x1="81.28" y1="53.34" x2="81.28" y2="48.26" width="0.1524" layer="91"/>
+<wire x1="68.58" y1="35.56" x2="78.74" y2="35.56" width="0.1524" layer="91"/>
+<wire x1="78.74" y1="35.56" x2="78.74" y2="50.8" width="0.1524" layer="91"/>
+<wire x1="78.74" y1="50.8" x2="86.36" y2="50.8" width="0.1524" layer="91"/>
 <label x="68.58" y="35.56" size="1.778" layer="95"/>
 <pinref part="U401" gate="G$1" pin="PB5(SCK)"/>
@@
 </segment>
 </net>
-<net name="N$7" class="0">
+<net name="TXLED1" class="0">
 <segment>
 <wire x1="111.76" y1="60.96" x2="106.68" y2="60.96" width="0.1524" layer="91"/>
@@
 </segment>
 </net>
-<net name="N$10" class="0">
+<net name="RXLED1" class="0">
 <segment>
 <wire x1="111.76" y1="58.42" x2="96.52" y2="58.42" width="0.1524" layer="91"/>
@@
 <net name="N$8" class="0">
 <segment>
-<wire x1="81.28" y1="38.1" x2="81.28" y2="35.56" width="0.1524" layer="91"/>
+<wire x1="86.36" y1="40.64" x2="86.36" y2="35.56" width="0.1524" layer="91"/>
 <pinref part="R001" gate="A" pin="1"/>
 <pinref part="D402" gate="G$1" pin="A"/>
@@
 </segment>
 </net>
+<net name="D0" class="0">
+<segment>
+<wire x1="-63.5" y1="99.06" x2="-73.66" y2="99.06" width="0.1524" layer="91"/>
+<label x="-73.66" y="99.06" size="1.778" layer="95"/>
+<pinref part="J002" gate="G$1" pin="1"/>
+</segment>
+<segment>
+<wire x1="68.58" y1="71.12" x2="76.2" y2="71.12" width="0.1524" layer="91"/>
+<wire x1="76.2" y1="71.12" x2="76.2" y2="86.36" width="0.1524" layer="91"/>
+<wire x1="76.2" y1="86.36" x2="83.82" y2="86.36" width="0.1524" layer="91"/>
+<label x="68.58" y="71.12" size="1.778" layer="95"/>
+<pinref part="U401" gate="G$1" pin="PD0(RXD)"/>
+<wire x1="93.98" y1="86.36" x2="111.76" y2="86.36" width="0.1524" layer="91"/>
+<pinref part="U001" gate="G$1" pin="TXD"/>
+<wire x1="83.82" y1="86.36" x2="93.98" y2="86.36" width="0" layer="91"/>
+</segment>
+</net>
+<net name="D1" class="0">
+<segment>
+<wire x1="-63.5" y1="96.52" x2="-73.66" y2="96.52" width="0.1524" layer="91"/>
+<label x="-73.66" y="96.52" size="1.778" layer="95"/>
+<pinref part="J002" gate="G$1" pin="2"/>
+</segment>
+<segment>
+<wire x1="68.58" y1="68.58" x2="78.74" y2="68.58" width="0.1524" layer="91"/>
+<wire x1="78.74" y1="68.58" x2="78.74" y2="83.82" width="0.1524" layer="91"/>
+<wire x1="78.74" y1="83.82" x2="83.82" y2="83.82" width="0.1524" layer="91"/>
+<label x="68.58" y="68.58" size="1.778" layer="95"/>
+<pinref part="U401" gate="G$1" pin="PD1(TXD)"/>
+<wire x1="93.98" y1="83.82" x2="111.76" y2="83.82" width="0.1524" layer="91"/>
+<pinref part="U001" gate="G$1" pin="RXD"/>
+<wire x1="83.82" y1="83.82" x2="93.98" y2="83.82" width="0" layer="91"/>
+</segment>
+</net>

Commit message: No regulator, with top labels
Parts:
- added S429: B3U-1000P, KwanSystems:B3U-1000P
- D001: value red -> blue
- D002: value green -> red
- D401: value blue -> green
- U001: device SparkFun:FT232RLSSOP -> SparkFun-DigitalIC:FT232RLSSOP
- U401: value ATMEGA168 -> ATMEGA328P; device SparkFun:ATMEGA168 -> SparkFun-DigitalIC:ATMEGA168
Connections:
- net D13: now also R001D.2; no longer R001A.2
- net GND: now also S429.1
- net N$11: now also R001B.1; no longer R001C.1
- net N$5: now also R001C.1; no longer R001D.1
- net N$8: now also R001D.1; no longer R001A.1
- net N$9: now also R001A.1; no longer R001B.1
- net RESET: now also S429.2
- net RXLED1: now also R001B.2; no longer R001C.2
- net TXLED1: now also R001A.2; no longer R001B.2
- net VCC: now also R001C.2; no longer R001D.2
Other:
- moved on the sheet: R001A, R001B, R001C, R001D
Changed lines of the file:
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@@
 </classes>
 <parts>
-<part name="U001" library="SparkFun" deviceset="FT232RL" device="SSOP"/>
+<part name="U001" library="SparkFun-DigitalIC" deviceset="FT232RL" device="SSOP"/>
 <part name="J001" library="KwanSystems" deviceset="USB_MICROB_JST" device=""/>
-<part name="U401" library="SparkFun" deviceset="ATMEGA168" device=""/>
+<part name="U401" library="SparkFun-DigitalIC" deviceset="ATMEGA168" device="" value="ATMEGA328P"/>
 <part name="C420" library="SparkFun" deviceset="CAP" device="0402-CAP" value="100nF"/>
 <part name="C404" library="SparkFun" deviceset="CAP" device="0402-CAP" value="100nF"/>
@@
 <part name="P+2" library="SparkFun" deviceset="VCC" device=""/>
 <part name="R001" library="KwanSystems" deviceset="RP4" device="04" value="680"/>
-<part name="D401" library="SparkFun-LED" deviceset="LED" device="0603" value="blue"/>
-<part name="D001" library="SparkFun-LED" deviceset="LED" device="0603" value="red"/>
-<part name="D002" library="SparkFun-LED" deviceset="LED" device="0603" value="green"/>
+<part name="D401" library="SparkFun-LED" deviceset="LED" device="0603" value="green"/>
+<part name="D001" library="SparkFun-LED" deviceset="LED" device="0603" value="blue"/>
+<part name="D002" library="SparkFun-LED" deviceset="LED" device="0603" value="red"/>
 <part name="D402" library="SparkFun-LED" deviceset="LED" device="0603" value="amber"/>
 <part name="P+3" library="SparkFun" deviceset="VCC" device=""/>
@@
 <part name="C408" library="SparkFun" deviceset="CAP" device="0402-CAP" value="18pF"/>
 <part name="Y401" library="KwanSystems" deviceset="CX2520" device="" value="16MHz"/>
+<part name="S429" library="KwanSystems" deviceset="B3U-1000P" device="" value=""/>
 </parts>
 <sheets>
@@
 <instance part="C017" gate="G$1" x="147.32" y="66.04"/>
 <instance part="P+2" gate="1" x="149.86" y="96.52"/>
-<instance part="R001" gate="D" x="-22.86" y="78.74" rot="R90"/>
-<instance part="R001" gate="B" x="106.68" y="45.72" rot="R90"/>
-<instance part="R001" gate="C" x="96.52" y="45.72" rot="R90"/>
-<instance part="R001" gate="A" x="86.36" y="45.72" rot="R90"/>
+<instance part="R001" gate="C" x="-22.86" y="78.74" rot="R90"/>
+<instance part="R001" gate="A" x="106.68" y="45.72" rot="R90"/>
+<instance part="R001" gate="B" x="96.52" y="45.72" rot="R90"/>
+<instance part="R001" gate="D" x="86.36" y="45.72" rot="R90"/>
 <instance part="D401" gate="G$1" x="-22.86" y="45.72"/>
 <instance part="D001" gate="G$1" x="96.52" y="33.02"/>
@@
 <instance part="Y401" gate="G$1" x="-5.08" y="55.88" rot="R90"/>
 <instance part="Y401" gate="G$2" x="-2.54" y="15.24"/>
+<instance part="S429" gate="S$1" x="-12.7" y="109.22" rot="R90"/>
 </instances>
 <busses>
@@
 <junction x="-12.7" y="48.26"/>
 <pinref part="Y401" gate="G$2" pin="1"/>
+<pinref part="S429" gate="S$1" pin="1"/>
+<wire x1="-12.7" y1="104.14" x2="-12.7" y2="83.82" width="0" layer="91"/>
+<junction x="-12.7" y="83.82"/>
 </segment>
 </net>
@@
 <pinref part="C404" gate="G$1" pin="1"/>
 <pinref part="C406" gate="G$1" pin="1"/>
-<pinref part="R001" gate="D" pin="2"/>
+<pinref part="R001" gate="C" pin="2"/>
 <pinref part="C418" gate="G$1" pin="1"/>
 <pinref part="R429" gate="G$1" pin="1"/>
@@
 <pinref part="U401" gate="G$1" pin="PC6(/RESET)"/>
 <pinref part="R429" gate="G$1" pin="2"/>
+<pinref part="S429" gate="S$1" pin="2"/>
+<wire x1="-12.7" y1="111.76" x2="12.7" y2="111.76" width="0" layer="91"/>
+<wire x1="12.7" y1="111.76" x2="12.7" y2="96.52" width="0" layer="91"/>
+<junction x="12.7" y="96.52"/>
 </segment>
 <segment>
@@
 <label x="68.58" y="35.56" size="1.778" layer="95"/>
 <pinref part="U401" gate="G$1" pin="PB5(SCK)"/>
-<pinref part="R001" gate="A" pin="2"/>
+<pinref part="R001" gate="D" pin="2"/>
 </segment>
 <segment>
@@
 <wire x1="106.68" y1="60.96" x2="106.68" y2="50.8" width="0.1524" layer="91"/>
 <pinref part="U001" gate="G$1" pin="TXLED"/>
-<pinref part="R001" gate="B" pin="2"/>
+<pinref part="R001" gate="A" pin="2"/>
 </segment>
 </net>
@@
 <wire x1="96.52" y1="58.42" x2="96.52" y2="50.8" width="0.1524" layer="91"/>
 <pinref part="U001" gate="G$1" pin="RXLED"/>
-<pinref part="R001" gate="C" pin="2"/>
+<pinref part="R001" gate="B" pin="2"/>
 </segment>
 </net>
@@
 <segment>
 <wire x1="96.52" y1="40.64" x2="96.52" y2="35.56" width="0.1524" layer="91"/>
+<pinref part="R001" gate="B" pin="1"/>
+<pinref part="D001" gate="G$1" pin="A"/>
+</segment>
+</net>
+<net name="N$5" class="0">
+<segment>
+<wire x1="-22.86" y1="73.66" x2="-22.86" y2="48.26" width="0.1524" layer="91"/>
 <pinref part="R001" gate="C" pin="1"/>
-<pinref part="D001" gate="G$1" pin="A"/>
-</segment>
-</net>
-<net name="N$5" class="0">
-<segment>
-<wire x1="-22.86" y1="73.66" x2="-22.86" y2="48.26" width="0.1524" layer="91"/>
+<pinref part="D401" gate="G$1" pin="A"/>
+</segment>
+</net>
+<net name="N$8" class="0">
+<segment>
+<wire x1="86.36" y1="40.64" x2="86.36" y2="35.56" width="0.1524" layer="91"/>
 <pinref part="R001" gate="D" pin="1"/>
-<pinref part="D401" gate="G$1" pin="A"/>
-</segment>
-</net>
-<net name="N$8" class="0">
-<segment>
-<wire x1="86.36" y1="40.64" x2="86.36" y2="35.56" width="0.1524" layer="91"/>
+<pinref part="D402" gate="G$1" pin="A"/>
+</segment>
+</net>
+<net name="N$9" class="0">
+<segment>
+<wire x1="106.68" y1="40.64" x2="106.68" y2="35.56" width="0.1524" layer="91"/>
 <pinref part="R001" gate="A" pin="1"/>
-<pinref part="D402" gate="G$1" pin="A"/>
-</segment>
-</net>
-<net name="N$9" class="0">
-<segment>
-<wire x1="106.68" y1="40.64" x2="106.68" y2="35.56" width="0.1524" layer="91"/>
-<pinref part="R001" gate="B" pin="1"/>
 <pinref part="D002" gate="G$1" pin="A"/>
 </segment>
