File: Precision Singleboard Charlieplex.brd (EAGLE design)
At the start: 76.2 x 76.2 mm, 265 parts, among them J402 EM406, J404 EM406, U401 ATMEGA328, U501 FT232RLSSOP, U602 ZF7, Y401 12.00

Commit message: Merged Mio's KwanSystems.lbr, updated all eagle files to use it.
Changed lines of the file:
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@@
 <?xml version="1.0" encoding="utf-8"?>
 <!DOCTYPE eagle SYSTEM "eagle.dtd">
-<eagle version="6.1">
+<eagle version="6.2">
 <drawing>
 <settings>
@@
 <contactref element="C407" pad="1"/>
 <contactref element="C408" pad="1"/>
-<contactref element="Y401" pad="2"/>
-<contactref element="Y401" pad="4"/>
+<contactref element="Y401" pad="2" route="any" routetag="1"/>
 <contactref element="J002" pad="4"/>
 <contactref element="C010" pad="2"/>
@@
 <wire x1="33.8074" y1="32.95" x2="33.8074" y2="31.35" width="0" layer="19" extent="1-1"/>
 <wire x1="32.092" y1="32.258" x2="33.8074" y2="32.95" width="0" layer="19" extent="1-1"/>
-<wire x1="32.042" y1="30.818" x2="32.092" y2="32.258" width="0" layer="19" extent="1-1"/>
-<wire x1="30.442" y1="28.618" x2="32.042" y2="30.818" width="0" layer="19" extent="1-1"/>
-<wire x1="30.392" y1="27.178" x2="30.442" y2="28.618" width="0" layer="19" extent="1-1"/>
 <wire x1="31.684" y1="36.322" x2="33.8074" y2="32.95" width="0" layer="19" extent="1-1"/>
+<wire x1="30.4292" y1="28.6258" x2="32.092" y2="32.258" width="0" layer="19" extent="1-1"/>
+<wire x1="30.392" y1="27.178" x2="30.4292" y2="28.6258" width="0" layer="19" extent="1-1"/>
 <wire x1="27.94" y1="39.37" x2="31.684" y2="36.322" width="0" layer="19" extent="1-1"/>
 <wire x1="37.775" y1="39.524" x2="31.684" y2="36.322" width="0" layer="19" extent="1-1"/>
@@
 <wire x1="34.29" y1="49.53" x2="35.175" y2="46.836" width="0" layer="19" extent="1-1"/>
 <wire x1="34.71" y1="51.816" x2="34.29" y2="49.53" width="0" layer="19" extent="1-1"/>
+<contactref element="Y401" pad="4" route="any" routetag="1"/>
 </signal>
 <signal name="VCC" class="1">
@@
 <contactref element="Y401" pad="1"/>
 <contactref element="U401" pad="7"/>
-<wire x1="30.442" y1="30.818" x2="33.8074" y2="29.75" width="0" layer="19" extent="1-1"/>
-<wire x1="30.392" y1="32.258" x2="30.442" y2="30.818" width="0" layer="19" extent="1-1"/>
+<wire x1="30.4292" y1="30.8102" x2="33.8074" y2="29.75" width="0" layer="19" extent="1-1"/>
+<wire x1="30.392" y1="32.258" x2="30.4292" y2="30.8102" width="0" layer="19" extent="1-1"/>
 </signal>
 <signal name="XTAL2">
@@
 <contactref element="Y401" pad="3"/>
 <contactref element="U401" pad="8"/>
-<wire x1="32.042" y1="28.618" x2="33.8074" y2="28.95" width="0" layer="19" extent="1-1"/>
-<wire x1="32.092" y1="27.178" x2="32.042" y2="28.618" width="0" layer="19" extent="1-1"/>
+<wire x1="32.0548" y1="28.6258" x2="33.8074" y2="28.95" width="0" layer="19" extent="1-1"/>
+<wire x1="32.092" y1="27.178" x2="32.0548" y2="28.6258" width="0" layer="19" extent="1-1"/>
 </signal>
 <signal name="P01">
@@
 </signal>
 </signals>
-<errors>
-</errors>
 </board>
 </drawing>
