File: Rocketometer2148 MPU6050.brd (EAGLE design)
At the start: 55.9 x 22.9 mm, 73 parts, among them J001 USB_MICROB_JST, J301 JST 2mm, J401 M07, J701 MICROSD-SOCKET, Q050 PMOS, U101 BMP180, U201 MIC5319, U301 MCP73831, U401 LPC2148, U601 MPU6050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

Commit message: In preparation for adding more resistor arrays to power supply
Parts:
- C461, C462: value 22pF -> 33pF
- U201: value MIC5319 -> 3.3V

Commit message: RocketometerMPU6050 as ordered
Parts:
- moved U$4 46.9 mm to (1.27, 7.62)
Connections:
- net N$11 renamed QWMG
- net N$3 renamed QWMB
- net N$9 renamed QWMR
- net PWMG: now also R402.8, U401.31; no longer R402.5, U401.33
- net PWMR: now also R402.5, U401.33; no longer R402.8, U401.31
Routing:
- net PWMR: track 18.5 -> 14.7 mm
- net PWMG: track 14.7 -> 18.5 mm
- net USB_ON: track 42.3 -> 41.0 mm
Changed lines of the file:
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@@
 <grid distance="10" unitdist="mil" unit="mil" style="lines" multiple="1" display="yes" altdistance="0.005" altunitdist="inch" altunit="inch"/>
 <layers>
-<layer number="1" name="Top" color="4" fill="1" visible="yes" active="yes"/>
+<layer number="1" name="Top" color="4" fill="1" visible="no" active="yes"/>
 <layer number="2" name="Route2" color="1" fill="3" visible="no" active="no"/>
 <layer number="3" name="Route3" color="4" fill="3" visible="no" active="no"/>
@@
 <attribute name="VALUE" x="13.843" y="2.4765" size="0.4064" layer="27" rot="R90"/>
 </element>
-<element name="U$4" library="KwanSystems" package="AXES" value="" x="47.752" y="1.016"/>
+<element name="U$4" library="KwanSystems" package="AXES" value="" x="1.27" y="7.62"/>
 <element name="JP3" library="SparkFun-Electromechanical" package="STAND-OFF-TIGHT" value="STAND-OFFTIGHT" x="15.24" y="11.43">
 <attribute name="DIGIKEY" value="$NOPART" x="15.24" y="11.43" size="1.778" layer="27" display="off"/>
@@
 <contactref element="U401" pad="58"/>
 <contactref element="S458" pad="P$1"/>
-<wire x1="41.402" y1="12.7" x2="41.656" y2="12.446" width="0.1524" layer="16"/>
-<wire x1="39.116" y1="12.7" x2="41.402" y2="12.7" width="0.1524" layer="16"/>
-<wire x1="35.306" y1="8.89" x2="39.116" y2="12.7" width="0.1524" layer="16"/>
+<wire x1="35.306" y1="8.89" x2="38.862" y2="12.446" width="0.1524" layer="16"/>
 <wire x1="35.306" y1="8.382" x2="35.306" y2="8.89" width="0.1524" layer="1"/>
 <wire x1="34.036" y1="7.112" x2="35.306" y2="8.382" width="0.1524" layer="1"/>
@@
 <via x="41.656" y="12.446" extent="1-16" drill="0.3302"/>
 <via x="35.306" y="8.89" extent="1-16" drill="0.3302"/>
-<wire x1="47.498" y1="16.002" x2="48.372" y2="16.002" width="0.1524" layer="16"/>
-<wire x1="47.244" y1="15.748" x2="47.498" y2="16.002" width="0.1524" layer="16"/>
-<wire x1="47.244" y1="15.24" x2="47.244" y2="15.748" width="0.1524" layer="16"/>
-<wire x1="47.498" y1="14.986" x2="47.244" y2="15.24" width="0.1524" layer="16"/>
 <via x="47.498" y="14.986" extent="1-16" drill="0.3302"/>
 <wire x1="42.418" y1="13.208" x2="48.006" y2="13.208" width="0.1524" layer="1"/>
@@
 <wire x1="48.006" y1="14.478" x2="47.498" y2="14.986" width="0.1524" layer="1"/>
 <wire x1="41.656" y1="12.446" x2="42.418" y2="13.208" width="0.1524" layer="1"/>
-<wire x1="23.622" y1="12.319" x2="23.622" y2="12.446" width="0.1524" layer="16"/>
-<wire x1="24.13" y1="11.811" x2="23.622" y2="12.319" width="0.1524" layer="16"/>
+<wire x1="24.13" y1="11.811" x2="23.417" y2="12.524" width="0.1524" layer="16"/>
 <wire x1="28.956" y1="11.811" x2="24.13" y2="11.811" width="0.1524" layer="16"/>
 <wire x1="29.972" y1="12.827" x2="28.956" y2="11.811" width="0.1524" layer="16"/>
 <wire x1="32.131" y1="12.827" x2="29.972" y2="12.827" width="0.1524" layer="16"/>
-<wire x1="33.655" y1="11.303" x2="32.131" y2="12.827" width="0.1524" layer="16"/>
-<wire x1="33.655" y1="9.017" x2="33.655" y2="11.303" width="0.1524" layer="16"/>
-<wire x1="33.401" y1="8.763" x2="33.655" y2="9.017" width="0.1524" layer="16"/>
+<wire x1="33.401" y1="11.557" x2="32.131" y2="12.827" width="0.1524" layer="16"/>
 <via x="33.401" y="8.763" extent="1-16" drill="0.3302"/>
-<wire x1="23.495" y1="12.573" x2="20.574" y2="12.573" width="0.1524" layer="16"/>
-<wire x1="23.622" y1="12.446" x2="23.495" y2="12.573" width="0.1524" layer="16"/>
-<wire x1="20.574" y1="12.573" x2="20.574" y2="12.524" width="0.1524" layer="16"/>
 <wire x1="34.036" y1="7.112" x2="33.401" y2="7.747" width="0.1524" layer="1"/>
 <wire x1="33.401" y1="7.747" x2="33.401" y2="8.763" width="0.1524" layer="1"/>
+<wire x1="33.401" y1="8.763" x2="33.401" y2="11.557" width="0.1524" layer="16"/>
+<wire x1="23.417" y1="12.524" x2="20.574" y2="12.524" width="0.1524" layer="16"/>
+<wire x1="48.372" y1="16.002" x2="47.498" y2="15.128" width="0.1524" layer="16"/>
+<wire x1="47.498" y1="15.128" x2="47.498" y2="14.986" width="0.1524" layer="16"/>
+<wire x1="41.656" y1="12.446" x2="38.862" y2="12.446" width="0.1524" layer="16"/>
 </signal>
 <signal name="CONN_D-">
@@
 <wire x1="33.274" y1="20.066" x2="31.75" y2="21.59" width="0.1524" layer="1"/>
 </signal>
-<signal name="PWMG">
-<contactref element="U401" pad="33"/>
-<contactref element="R402" pad="5"/>
-<wire x1="27.674" y1="14.418" x2="27.674" y2="15.494" width="0.1524" layer="1"/>
-<wire x1="27.674" y1="15.494" x2="27.686" y2="15.494" width="0.1524" layer="1"/>
-<via x="27.686" y="15.494" extent="1-16" drill="0.3302"/>
-<wire x1="27.686" y1="15.494" x2="25.146" y2="15.494" width="0.1524" layer="16"/>
-<wire x1="25.146" y1="15.494" x2="20.828" y2="19.812" width="0.1524" layer="16"/>
-<wire x1="20.828" y1="19.812" x2="17.78" y2="19.812" width="0.1524" layer="16"/>
-<wire x1="17.78" y1="19.812" x2="17.018" y2="20.574" width="0.1524" layer="16"/>
-<wire x1="17.018" y1="20.574" x2="16.261" y2="20.574" width="0.1524" layer="16"/>
-<wire x1="16.261" y1="20.574" x2="16.248" y2="20.612" width="0.1524" layer="16"/>
-</signal>
 <signal name="COMPINT">
 <contactref element="U801" pad="15"/>
@@
 <wire x1="43.876" y1="8.382" x2="45.497" y2="8.382" width="0.1524" layer="16"/>
 </signal>
-<signal name="N$9">
+<signal name="QWMR">
 <contactref element="R402" pad="4"/>
 <contactref element="D401" pad="2"/>
@@
 <wire x1="14.212" y1="21.348" x2="14.212" y2="21.562" width="0.1524" layer="16"/>
 </signal>
-<signal name="N$11">
+<signal name="QWMG">
 <contactref element="R402" pad="1"/>
 <contactref element="D401" pad="3"/>
@@
 <wire x1="14.478" y1="18.328" x2="14.212" y2="18.062" width="0.1524" layer="16"/>
 </signal>
-<signal name="N$3">
+<signal name="QWMB">
 <contactref element="R402" pad="2"/>
 <contactref element="D401" pad="4"/>
@@
 </signal>
 <signal name="PWMR">
-<contactref element="R402" pad="8"/>
-<contactref element="U401" pad="31"/>
-<wire x1="16.248" y1="19.012" x2="17.056" y2="19.012" width="0.1524" layer="16"/>
-<wire x1="17.056" y1="19.012" x2="17.272" y2="18.796" width="0.1524" layer="16"/>
-<wire x1="17.272" y1="18.796" x2="20.066" y2="18.796" width="0.1524" layer="16"/>
-<wire x1="20.066" y1="18.796" x2="25.654" y2="13.208" width="0.1524" layer="16"/>
-<wire x1="25.654" y1="13.208" x2="28.702" y2="13.208" width="0.1524" layer="16"/>
-<wire x1="28.702" y1="13.208" x2="29.718" y2="14.224" width="0.1524" layer="16"/>
-<via x="29.718" y="14.224" extent="1-16" drill="0.3302"/>
-<wire x1="29.718" y1="14.224" x2="30.024" y2="14.53" width="0.1524" layer="1"/>
-<wire x1="30.024" y1="14.53" x2="30.024" y2="16.268" width="0.1524" layer="1"/>
+<contactref element="U401" pad="33"/>
+<contactref element="R402" pad="5"/>
+<wire x1="27.674" y1="14.418" x2="27.674" y2="15.494" width="0.1524" layer="1"/>
+<wire x1="27.674" y1="15.494" x2="27.686" y2="15.494" width="0.1524" layer="1"/>
+<via x="27.686" y="15.494" extent="1-16" drill="0.3302"/>
+<wire x1="27.686" y1="15.494" x2="25.146" y2="15.494" width="0.1524" layer="16"/>
+<wire x1="25.146" y1="15.494" x2="20.828" y2="19.812" width="0.1524" layer="16"/>
+<wire x1="20.828" y1="19.812" x2="17.78" y2="19.812" width="0.1524" layer="16"/>
+<wire x1="17.78" y1="19.812" x2="17.018" y2="20.574" width="0.1524" layer="16"/>
+<wire x1="17.018" y1="20.574" x2="16.261" y2="20.574" width="0.1524" layer="16"/>
+<wire x1="16.261" y1="20.574" x2="16.248" y2="20.612" width="0.1524" layer="16"/>
 </signal>
 <signal name="RESET" class="1">
@@
 <wire x1="15.819" y1="3.556" x2="15.819" y2="4.856" width="0.1524" layer="1"/>
 </signal>
+<signal name="PWMG">
+<contactref element="R402" pad="8"/>
+<contactref element="U401" pad="31"/>
+<wire x1="16.248" y1="19.012" x2="17.056" y2="19.012" width="0.1524" layer="16"/>
+<wire x1="17.056" y1="19.012" x2="17.272" y2="18.796" width="0.1524" layer="16"/>
+<wire x1="17.272" y1="18.796" x2="20.066" y2="18.796" width="0.1524" layer="16"/>
+<wire x1="20.066" y1="18.796" x2="25.654" y2="13.208" width="0.1524" layer="16"/>
+<wire x1="25.654" y1="13.208" x2="28.702" y2="13.208" width="0.1524" layer="16"/>
+<wire x1="28.702" y1="13.208" x2="29.718" y2="14.224" width="0.1524" layer="16"/>
+<via x="29.718" y="14.224" extent="1-16" drill="0.3302"/>
+<wire x1="29.718" y1="14.224" x2="30.024" y2="14.53" width="0.1524" layer="1"/>
+<wire x1="30.024" y1="14.53" x2="30.024" y2="16.268" width="0.1524" layer="1"/>
+</signal>
 </signals>

Commit message: Added KwanAstro after the little crash of 2012
Parts:
- removed Q050: PMOS, SparkFun:SOT23-3
- added Q001: PMOS, SparkFun-DiscreteSemi:SOT23-3
Connections:
- net N$6: now also Q001.3; no longer Q050.3
- net USB_LIGHT: now also Q001.1; no longer Q050.1
- net VCC: now also Q001.2; no longer Q050.2
Routing:
- net N$6: track 26.4 -> 25.3 mm
Changed lines of the file:
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@@
 <attribute name="DIGIKEY" value="350-2037-1-ND" x="49.022" y="20.574" size="1.778" layer="28" rot="MR270" display="off"/>
-</element>
-<element name="Q050" library="SparkFun" package="SOT23-3" value="PMOS" x="49.022" y="19.558" smashed="yes">
-<attribute name="NAME" x="48.1965" y="19.304" size="0.4064" layer="51"/>
-<attribute name="VALUE" x="48.006" y="19.3675" size="0.4064" layer="27"/>
-<attribute name="LOGO_3D50" value="NOLOGO" x="49.022" y="19.558" size="1.778" layer="22" display="off"/>
-<attribute name="DIGIKEY" value="NTR1P02T1GOSCT-ND" x="49.022" y="19.558" size="1.778" layer="27" display="off"/>
 </element>
 <element name="J001" library="KwanSystems" package="UB-MC5BR3-SD204-4S" value="USB_MICROB_JST" x="54.356" y="11.43" rot="MR270">
@@
 <element name="U$1" library="KwanSystems" package="KWAN_ACC" value="" x="7.62" y="11.43"/>
 <element name="U$6" library="KwanSystems" package="OSHW_ACC" value="" x="8.89" y="3.556" rot="MR0"/>
+<element name="Q001" library="SparkFun-DiscreteSemi" package="SOT23-3" value="PMOS" x="-2.032" y="-1.016"/>
 </elements>
 <signals>
@@
 <contactref element="U801" pad="2"/>
 <contactref element="C802" pad="1"/>
-<contactref element="Q050" pad="2"/>
 <contactref element="U201" pad="5"/>
 <contactref element="C215" pad="1"/>
@@
 <wire x1="30.861" y1="2.936" x2="30.524" y2="3.273" width="0.1524" layer="1"/>
 <wire x1="30.524" y1="3.273" x2="30.524" y2="5.068" width="0.1524" layer="1"/>
-<wire x1="49.972" y1="18.558" x2="49.784" y2="18.37" width="0.1524" layer="1" curve="90"/>
 <wire x1="49.784" y1="18.37" x2="49.784" y2="17.018" width="0.1524" layer="1"/>
 <wire x1="49.784" y1="17.018" x2="49.672" y2="17.018" width="0.1524" layer="1"/>
@@
 <wire x1="30.524" y1="6.984" x2="30.734" y2="7.194" width="0.1524" layer="1"/>
 <wire x1="30.734" y1="7.194" x2="30.734" y2="8.89" width="0.1524" layer="1"/>
+<contactref element="Q001" pad="2"/>
+<wire x1="-1.082" y1="-2.016" x2="6.87" y2="3.806" width="0" layer="19" extent="1-1"/>
 </signal>
 <signal name="GND" class="1">
@@
 </signal>
 <signal name="USB_LIGHT">
-<contactref element="Q050" pad="1"/>
 <contactref element="R051" pad="2"/>
 <contactref element="U401" pad="17"/>
-<wire x1="48.072" y1="18.558" x2="48.26" y2="18.558" width="0.1524" layer="1"/>
 <wire x1="48.26" y1="18.558" x2="48.26" y2="17.018" width="0.1524" layer="1"/>
 <wire x1="48.26" y1="17.018" x2="48.372" y2="17.018" width="0.1524" layer="1"/>
@@
 <wire x1="37.024" y1="16.764" x2="48.372" y2="16.764" width="0.1524" layer="1"/>
 <wire x1="48.372" y1="16.764" x2="48.372" y2="17.018" width="0.1524" layer="1"/>
+<contactref element="Q001" pad="1"/>
+<wire x1="-2.982" y1="-2.016" x2="37.024" y2="16.268" width="0" layer="19" extent="1-1"/>
 </signal>
 <signal name="N$6">
 <contactref element="D050" pad="A"/>
 <contactref element="R031" pad="1"/>
-<contactref element="Q050" pad="3"/>
-<wire x1="49.022" y1="20.658" x2="49.022" y2="19.558" width="0.1524" layer="1"/>
 <via x="49.022" y="19.558" extent="1-16" drill="0.3302"/>
 <wire x1="49.022" y1="19.558" x2="49.022" y2="20.574" width="0.1524" layer="16"/>
@@
 <wire x1="53.086" y1="6.35" x2="53.086" y2="17.26" width="0.1524" layer="16"/>
 <wire x1="53.086" y1="17.26" x2="49.772" y2="20.574" width="0.1524" layer="16"/>
+<contactref element="Q001" pad="3"/>
+<wire x1="-2.032" y1="0.084" x2="47.752" y2="6.35" width="0" layer="19" extent="1-16"/>
 </signal>
 <signal name="N$7">
@@
 </signal>
 </signals>
-<errors>
-</errors>
 </board>
 </drawing>

Commit message: As (attempted to be) flown 23 Feb 2013
Parts:
- moved Q001 55.0 mm to (49.0, 19.6)
Connections:
- new net SCL1: U601.7
- new net SDA1: U601.6
Changed lines of the file:
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@@
 <?xml version="1.0" encoding="utf-8"?>
 <!DOCTYPE eagle SYSTEM "eagle.dtd">
-<eagle version="6.2">
+<eagle version="6.3">
 <drawing>
 <settings>
@@
 <grid distance="10" unitdist="mil" unit="mil" style="lines" multiple="1" display="yes" altdistance="0.005" altunitdist="inch" altunit="inch"/>
 <layers>
-<layer number="1" name="Top" color="4" fill="1" visible="no" active="yes"/>
+<layer number="1" name="Top" color="4" fill="1" visible="yes" active="yes"/>
 <layer number="2" name="Route2" color="1" fill="3" visible="no" active="no"/>
 <layer number="3" name="Route3" color="4" fill="3" visible="no" active="no"/>
@@
 </class>
 </classes>
-<designrules>
+<designrules name="default">
 <description language="de">&lt;b&gt;EAGLE Design Rules&lt;/b&gt;
 &lt;p&gt;
@@
 <element name="U$1" library="KwanSystems" package="KWAN_ACC" value="" x="7.62" y="11.43"/>
 <element name="U$6" library="KwanSystems" package="OSHW_ACC" value="" x="8.89" y="3.556" rot="MR0"/>
-<element name="Q001" library="SparkFun-DiscreteSemi" package="SOT23-3" value="PMOS" x="-2.032" y="-1.016"/>
+<element name="Q001" library="SparkFun-DiscreteSemi" package="SOT23-3" value="PMOS" x="49.022" y="19.558"/>
 </elements>
 <signals>
@@
 <wire x1="30.734" y1="7.194" x2="30.734" y2="8.89" width="0.1524" layer="1"/>
 <contactref element="Q001" pad="2"/>
-<wire x1="-1.082" y1="-2.016" x2="6.87" y2="3.806" width="0" layer="19" extent="1-1"/>
+<wire x1="49.972" y1="18.558" x2="49.784" y2="18.558" width="0.4064" layer="1"/>
+<wire x1="49.784" y1="18.558" x2="49.784" y2="18.37" width="0.4064" layer="1"/>
 </signal>
 <signal name="GND" class="1">
@@
 <wire x1="48.372" y1="16.764" x2="48.372" y2="17.018" width="0.1524" layer="1"/>
 <contactref element="Q001" pad="1"/>
-<wire x1="-2.982" y1="-2.016" x2="37.024" y2="16.268" width="0" layer="19" extent="1-1"/>
+<wire x1="48.26" y1="18.558" x2="48.072" y2="18.558" width="0.4064" layer="1"/>
 </signal>
 <signal name="N$6">
@@
 <wire x1="53.086" y1="17.26" x2="49.772" y2="20.574" width="0.1524" layer="16"/>
 <contactref element="Q001" pad="3"/>
-<wire x1="-2.032" y1="0.084" x2="47.752" y2="6.35" width="0" layer="19" extent="1-16"/>
+<wire x1="49.022" y1="20.574" x2="49.022" y2="20.658" width="0" layer="19" extent="1-16"/>
 </signal>
 <signal name="N$7">
@@
 <wire x1="30.024" y1="14.53" x2="30.024" y2="16.268" width="0.1524" layer="1"/>
 </signal>
+<signal name="SDA1">
+<contactref element="U601" pad="6"/>
+</signal>
+<signal name="SCL1">
+<contactref element="U601" pad="7"/>
+</signal>
 </signals>
