File: Rocketometer2148 MPU6050.brd (EAGLE design)
At the start: 55.9 x 22.9 mm, 73 parts, among them J001 USB_MICROB_JST, J301 JST 2mm, J401 M07, J701 MICROSD-SOCKET, Q001 PMOS, U101 BMP180, U201 3.3V, U301 MCP73831, U401 LPC2148, U601 MPU6050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

Commit message: moved PEG from work to Kwan workspace
Parts:
- removed U$1: (no value), KwanSystems:KWAN_ACC
- U601: value MPU6050 -> MPU9150; device KwanSystems:MPU60X0 -> KwanSystems:LLGA24
- moved C610 0.25 mm to (8.89, 7.87)
Connections:
- removed net SCL1: U601.7
- removed net SDA1: U601.6
- net GND: now also U601.15, U601.17
- net VCC: now also U601.3
Routing:
- net VCC: track 165.3 -> 167.9 mm
- net N$6: track 25.3 -> 26.4 mm
Other:
- board text added: "v2.0 4 Oct 2013"
- board text removed: "v1.0 19 Nov 2012"
Changed lines of the file:
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@@
 <?xml version="1.0" encoding="utf-8"?>
 <!DOCTYPE eagle SYSTEM "eagle.dtd">
-<eagle version="6.3">
+<eagle version="6.2">
 <drawing>
 <settings>
@@
 <layer number="23" name="tOrigins" color="15" fill="1" visible="yes" active="yes"/>
 <layer number="24" name="bOrigins" color="15" fill="1" visible="yes" active="yes"/>
-<layer number="25" name="tNames" color="13" fill="1" visible="yes" active="yes"/>
-<layer number="26" name="bNames" color="13" fill="1" visible="yes" active="yes"/>
+<layer number="25" name="tNames" color="13" fill="1" visible="no" active="yes"/>
+<layer number="26" name="bNames" color="13" fill="1" visible="no" active="yes"/>
 <layer number="27" name="tValues" color="7" fill="1" visible="no" active="yes"/>
 <layer number="28" name="bValues" color="7" fill="1" visible="no" active="yes"/>
@@
 <layer number="50" name="dxf" color="7" fill="1" visible="no" active="yes"/>
 <layer number="51" name="tDocu" color="11" fill="1" visible="yes" active="yes"/>
-<layer number="52" name="bDocu" color="3" fill="1" visible="no" active="yes"/>
+<layer number="52" name="bDocu" color="3" fill="1" visible="yes" active="yes"/>
 <layer number="53" name="tGND_GNDA" color="7" fill="9" visible="no" active="no"/>
 <layer number="54" name="bGND_GNDA" color="1" fill="9" visible="no" active="no"/>
@@
 <text x="30.099" y="19.304" size="0.8128" layer="22" rot="MR0">GND</text>
 <text x="39.116" y="0.381" size="1.27" layer="22" rot="MR0">RocketometerMPU6050</text>
-<text x="43.942" y="5.715" size="0.8128" layer="21">v1.0 19 Nov 2012</text>
+<text x="43.942" y="5.715" size="0.8128" layer="21">v2.0 4 Oct 2013</text>
 <text x="19.05" y="6.477" size="0.8128" layer="22" rot="MR0">St Kwan's Home for</text>
 <text x="19.05" y="5.461" size="0.8128" layer="22" rot="MR0">the Terminally ADD</text>
@@
 </class>
 </classes>
-<designrules name="default">
+<designrules>
 <description language="de">&lt;b&gt;EAGLE Design Rules&lt;/b&gt;
 &lt;p&gt;
@@
 <attribute name="DIGIKEY" value="445-7395-1-ND" x="9.398" y="21.082" size="1.778" layer="27" rot="R90" display="off"/>
 </element>
-<element name="C610" library="SparkFun" package="0402-CAP" value="100nF" x="8.89" y="7.62" smashed="yes">
-<attribute name="NAME" x="9.525" y="7.3025" size="0.4064" layer="51"/>
-<attribute name="VALUE" x="7.8105" y="6.477" size="0.4064" layer="27"/>
-<attribute name="DIGIKEY" value="445-1265-1-ND" x="8.89" y="7.62" size="1.778" layer="27" display="off"/>
+<element name="C610" library="SparkFun" package="0402-CAP" value="100nF" x="8.89" y="7.874" smashed="yes">
+<attribute name="NAME" x="9.525" y="7.5565" size="0.4064" layer="51"/>
+<attribute name="VALUE" x="7.8105" y="6.731" size="0.4064" layer="27"/>
+<attribute name="DIGIKEY" value="445-1265-1-ND" x="8.89" y="7.874" size="1.778" layer="27" display="off"/>
 </element>
 <element name="C613" library="SparkFun" package="0402-CAP" value="100nF" x="11.176" y="10.922" smashed="yes" rot="R270">
@@
 <attribute name="VALUE" x="14.1605" y="5.207" size="0.4064" layer="27"/>
 </element>
-<element name="U601" library="KwanSystems" package="MPU60X0" value="MPU6050" x="7.62" y="11.43" smashed="yes">
-<attribute name="LOGO_3D50" value="NOLOGO" x="7.62" y="11.43" size="1.778" layer="21" display="off"/>
-<attribute name="NAME" x="6.096" y="12.192" size="0.8128" layer="51"/>
-<attribute name="VALUE" x="10.16" y="10.16" size="0.8128" layer="27"/>
-<attribute name="DIGIKEY" value="$NOPART" x="7.62" y="11.43" size="1.778" layer="27" display="off"/>
-</element>
 <element name="U$5" library="KwanSystems" package="KWAN_ACC" value="" x="7.62" y="11.43" rot="MR0"/>
-<element name="U$1" library="KwanSystems" package="KWAN_ACC" value="" x="7.62" y="11.43"/>
 <element name="U$6" library="KwanSystems" package="OSHW_ACC" value="" x="8.89" y="3.556" rot="MR0"/>
 <element name="Q001" library="SparkFun-DiscreteSemi" package="SOT23-3" value="PMOS" x="49.022" y="19.558"/>
+<element name="U601" library="KwanSystems" package="LLGA24" value="MPU9150" x="7.62" y="11.43" smashed="yes">
+<attribute name="NAME" x="6.604" y="11.938" size="0.6096" layer="51"/>
+<attribute name="VALUE" x="10.16" y="10.16" size="1.27" layer="27"/>
+</element>
 </elements>
 <signals>
@@
 <contactref element="C908" pad="1"/>
 <contactref element="C907" pad="1"/>
-<contactref element="U601" pad="13"/>
-<contactref element="U601" pad="8"/>
 <contactref element="J401" pad="8"/>
 <wire x1="27.674" y1="9.418" x2="25.654" y2="9.418" width="0.1524" layer="1"/>
@@
 <wire x1="5.334" y1="20.432" x2="5.334" y2="19.05" width="0.1524" layer="1"/>
 <wire x1="5.334" y1="19.05" x2="3.048" y2="16.764" width="0.1524" layer="1"/>
-<wire x1="3.048" y1="16.764" x2="3.048" y2="8.636" width="0.1524" layer="1"/>
+<wire x1="3.048" y1="16.764" x2="3.048" y2="11.684" width="0.1524" layer="1"/>
+<wire x1="3.048" y1="11.68" x2="3.048" y2="8.636" width="0.1524" layer="1"/>
 <wire x1="3.048" y1="8.636" x2="5.334" y2="8.636" width="0.1524" layer="1"/>
 <wire x1="5.334" y1="8.636" x2="6.87" y2="8.636" width="0.1524" layer="1"/>
@@
 <wire x1="49.972" y1="18.558" x2="49.784" y2="18.558" width="0.4064" layer="1"/>
 <wire x1="49.784" y1="18.558" x2="49.784" y2="18.37" width="0.4064" layer="1"/>
+<contactref element="U601" pad="13"/>
+<contactref element="U601" pad="3"/>
+<contactref element="U601" pad="8"/>
+<wire x1="5.62" y1="11.68" x2="3.048" y2="11.68" width="0.1524" layer="1"/>
+<wire x1="3.048" y1="11.68" x2="3.048" y2="11.684" width="0.1524" layer="1"/>
 </signal>
 <signal name="GND" class="1">
@@
 <contactref element="Y401" pad="4" route="any" routetag="1"/>
 <contactref element="C613" pad="1"/>
-<contactref element="C610" pad="2"/>
 <contactref element="C620" pad="1"/>
 <contactref element="C449" pad="1"/>
@@
 <contactref element="C907" pad="2"/>
 <contactref element="U902" pad="7"/>
-<contactref element="U601" pad="18"/>
-<contactref element="U601" pad="18"/>
-<contactref element="U601" pad="11"/>
-<contactref element="U601" pad="1"/>
-<contactref element="U601" pad="9"/>
 <polygon width="0.1524" layer="1" thermals="no">
 <vertex x="2.54" y="22.86"/>
@@
 <via x="47.244" y="11.43" extent="1-16" drill="0.3302"/>
 <via x="16.51" y="17.526" extent="1-16" drill="0.3302"/>
-<via x="10.414" y="8.128" extent="1-16" drill="0.3302"/>
 <via x="3.81" y="14.478" extent="1-16" drill="0.3302"/>
 <via x="12.7" y="6.477" extent="1-16" drill="0.3302"/>
@@
 <via x="4.826" y="0.889" extent="1-16" drill="0.3302"/>
 <via x="28.702" y="6.096" extent="1-16" drill="0.3302"/>
+<contactref element="U601" pad="18"/>
+<contactref element="U601" pad="17"/>
+<contactref element="U601" pad="15"/>
+<contactref element="U601" pad="9"/>
+<contactref element="U601" pad="1"/>
+<contactref element="U601" pad="11"/>
+<contactref element="C610" pad="2"/>
 </signal>
 <signal name="VLIPO">
@@
 <wire x1="53.086" y1="17.26" x2="49.772" y2="20.574" width="0.1524" layer="16"/>
 <contactref element="Q001" pad="3"/>
-<wire x1="49.022" y1="20.574" x2="49.022" y2="20.658" width="0" layer="19" extent="1-16"/>
+<wire x1="49.022" y1="20.658" x2="49.022" y2="19.558" width="0.1524" layer="1"/>
 </signal>
 <signal name="N$7">
@@
 <contactref element="J401" pad="7"/>
 <contactref element="U902" pad="2"/>
-<contactref element="U601" pad="24"/>
 <wire x1="23.36" y1="18.284" x2="23.335" y2="18.288" width="0.1524" layer="1"/>
 <wire x1="23.335" y1="18.288" x2="22.86" y2="18.288" width="0.1524" layer="1"/>
@@
 <wire x1="13.081" y1="10.541" x2="13.081" y2="14.605" width="0.1524" layer="1"/>
 <wire x1="13.081" y1="14.605" x2="11.938" y2="15.748" width="0.1524" layer="1"/>
+<contactref element="U601" pad="24"/>
 </signal>
 <signal name="SCL0">
@@
 <contactref element="J401" pad="6"/>
 <contactref element="U902" pad="1"/>
-<contactref element="U601" pad="23"/>
 <wire x1="23.36" y1="18.834" x2="23.335" y2="20.795" width="0.1524" layer="1"/>
 <wire x1="23.335" y1="20.795" x2="24.13" y2="21.59" width="0.1524" layer="1"/>
@@
 <wire x1="4.572" y1="16.002" x2="6.35" y2="16.002" width="0.1524" layer="1"/>
 <wire x1="6.35" y1="16.002" x2="6.604" y2="15.748" width="0.1524" layer="1"/>
+<contactref element="U601" pad="23"/>
 </signal>
 <signal name="ACCINT">
-<contactref element="U601" pad="12"/>
 <contactref element="U401" pad="47"/>
 <via x="11.684" y="8.509" extent="1-16" drill="0.3302"/>
@@
 <wire x1="8.87" y1="9.271" x2="10.922" y2="9.271" width="0.1524" layer="1"/>
 <wire x1="10.922" y1="9.271" x2="11.684" y2="8.509" width="0.1524" layer="1"/>
+<contactref element="U601" pad="12"/>
 </signal>
 <signal name="RX0">
@@
 <signal name="N$13">
 <contactref element="C610" pad="1"/>
+<wire x1="8.24" y1="7.874" x2="7.87" y2="7.99" width="0.1524" layer="1"/>
+<wire x1="7.87" y1="7.99" x2="7.87" y2="9.455" width="0.1524" layer="1"/>
 <contactref element="U601" pad="10"/>
-<wire x1="8.24" y1="7.62" x2="7.87" y2="7.99" width="0.1524" layer="1"/>
-<wire x1="7.87" y1="7.99" x2="7.87" y2="9.455" width="0.1524" layer="1"/>
 </signal>
 <signal name="N$1">
 <contactref element="C620" pad="2"/>
-<contactref element="U601" pad="20"/>
 <wire x1="8.37" y1="13.405" x2="8.37" y2="14.602" width="0.1524" layer="1"/>
 <wire x1="8.37" y1="14.602" x2="8.24" y2="14.732" width="0.1524" layer="1"/>
+<contactref element="U601" pad="20"/>
 </signal>
 <signal name="XACC">
@@
 <wire x1="30.024" y1="14.53" x2="30.024" y2="16.268" width="0.1524" layer="1"/>
 </signal>
-<signal name="SDA1">
-<contactref element="U601" pad="6"/>
-</signal>
-<signal name="SCL1">
-<contactref element="U601" pad="7"/>
-</signal>
 </signals>
+<errors>
+</errors>
 </board>
 </drawing>

Commit message: New version of rocketometer board for production
Parts:
- added C001: 4.7uF, SparkFun:0402-CAP
- added C002: 100nF, SparkFun-Passives:0402-CAP
- added D402: SMLP36RGB2W(R), KwanSystems:SMLP36
- added U903: MCP1525, KwanSystems:SOT-23-3
Connections:
- new net N$10: C001.1, U902.5, U903.2
- net GND: now also C001.2, C002.2, U903.3
- net QWMB: now also D402.1
- net QWMG: now also D402.3
- net QWMR: now also D402.5
- net VCC: now also C002.1, D402.2, D402.4, D402.6, U903.1
Routing:
- net VCC: track 167.9 -> 0.00 mm, vias 4 -> 0
- net SDA0: track 68.7 -> 0.00 mm, vias 5 -> 0
- net SCL0: track 68.4 -> 0.00 mm, vias 6 -> 0
- net VLIPO: track 57.1 -> 0.00 mm, vias 6 -> 0
- net USB_ON: track 41.0 -> 0.00 mm, vias 4 -> 0
- net VBUS: track 36.5 -> 0.00 mm
- net COMPINT: track 30.2 -> 0.00 mm, vias 2 -> 0
- net RESET: track 28.3 -> 0.00 mm, vias 2 -> 0
- net N$6: track 26.4 -> 0.00 mm, vias 1 -> 0
- net ACCINT: track 19.8 -> 0.00 mm, vias 2 -> 0
- net VIN: track 19.4 -> 0.00 mm
- net PWMG: track 18.5 -> 0.00 mm, vias 1 -> 0
- net ZACC: track 16.4 -> 0.00 mm, vias 2 -> 0
- net BSL: track 16.2 -> 0.00 mm, vias 1 -> 0
- net USBD+: track 14.8 -> 0.00 mm, vias 1 -> 0
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Other:
- board text added: "0.1 inch grid"
- board text added: "All holes 0.12 inch diameter - accept #4 Philipps screw"
- board text added: "v2.0 15 May 2013"
- board text removed: "v2.0 4 Oct 2013"
