File: Precision ATMega32U4.sch (EAGLE design)
At the start: 157 parts, among them U201 5319, Y401 16MHz

Commit message: Started RocketometerATMega.sch, finished PrecisionATMega32U4
Parts:
- removed C003, C424: 1uF, SparkFun:CAP0603-CAP
- removed C414: 4.7uF, SparkFun:CAP0603-CAP
- removed C420: 100nF, SparkFun:CAP0603-CAP
- removed R6: 1M, SparkFun:RESISTOR0603-RES
- removed U$1: ATMEGA32U4TQFP, SparkFun-DigitalIC:ATMEGA32U4TQFP
- removed Z1, Z2: CG0603MLC-05E, varistor:VARISTORCN0603
- added C406: 1uF, SparkFun:CAP0603-CAP
- added U401: ATMEGA32U4TQFP, SparkFun-DigitalIC:ATMEGA32U4TQFP
- R7: device KwanSystems:RP2EXB24V -> SparkFun-Passives:RESISTOR0603-RES
Connections:
- removed net AREF: C420.1, U$1.AREF
- net AT_RX: now also U401.PD2(RX); no longer U$1.PD2(RX)
- net AT_TX: now also U401.PD3(TX); no longer U$1.PD3(TX)
- net D+: no longer Z1.1
- net D-: no longer Z2.1
- net GND: now also C406.2, R7.1, U401.GND@15, U401.GND@23, U401.GND@35, U401.GND@43, U401.UGND; no longer C003.2, C414.1, C420.2, C424.2, R7B.1, U$1.GND@15, U$1.GND@23, U$1.GND@35, U$1.GND@43, U$1.UGND, Z1.2, Z2.2
- net HWB: now also R7.2, U401.PE2/!HWB; no longer R7B.2, U$1.PE2/!HWB
- net MISO: now also U401.PB3(MISO); no longer U$1.PB3(MISO)
- net MOSI: now also U401.PB2(MOSI); no longer U$1.PB2(MOSI)
- net P01: now also U401.PF7(ADC7); no longer U$1.PF7(ADC7)
- net P02: now also U401.PC7; no longer U$1.PC7
- net P03: now also U401.PC6; no longer U$1.PC6
- net P04: now also U401.PB6(ADC13); no longer U$1.PB6(ADC13)
- net P05: now also U401.PB5(ADC12); no longer U$1.PB5(ADC12)
- net P06: now also U401.PB4(ADC11); no longer U$1.PB4(ADC11)
- net P07: now also U401.PD7(ADC10); no longer U$1.PD7(ADC10)
- net P08: now also U401.PD4(ADC8); no longer U$1.PD4(ADC8)
- net P09: now also U401.PD0(SCL); no longer U$1.PD0(SCL)
- net P10: now also U401.PB7; no longer U$1.PB7
- net P11: now also U401.PF0(ADC0); no longer U$1.PF4(ADC4)
- net P12: now also U401.PE6; no longer U$1.PE6
- net P13: now also U401.PF1(ADC1); no longer U$1.PF1(ADC1)
- net P14: now also U401.PF4(ADC4); no longer U$1.PF6(ADC6)
- net P15: now also U401.PF5(ADC5); no longer U$1.PF0(ADC0)
- net P16: now also U401.PF6(ADC6); no longer U$1.PF5(ADC5)
- net PPS: now also U401.PD1(SDA); no longer U$1.PD1(SDA)
- net RD+: now also U401.D+; no longer U$1.D+
- net RD-: now also U401.D-; no longer U$1.D-
- net RESET: now also U401.!RESET; no longer R7A.2, U$1.!RESET
- net RXLED: now also U401.PB0(SS); no longer U$1.PB0(SS)
- net SCK: now also U401.PB1(SCK); no longer U$1.PB1(SCK)
- net TXLED: now also U401.PD5; no longer U$1.PD5
- net UCAP: now also C406.1, U401.UCAP; no longer C003.1, U$1.UCAP
- net VCC: now also U401.AREF, U401.AVCC@24, U401.AVCC@44, U401.UVCC, U401.VBUS, U401.VCC@14, U401.VCC@34; no longer C414.2, C424.1, R7A.1, U$1.AVCC@24, U$1.AVCC@44, U$1.UVCC, U$1.VBUS, U$1.VCC@14, U$1.VCC@34
- net XTAL1: now also U401.XTAL1; no longer R6.2, U$1.XTAL1
- net XTAL2: now also U401.XTAL2; no longer R6.1, U$1.XTAL2
Other:
- note removed: "Arduino LEONARDO"
- note removed: "TM"
- note removed: "USB"
- moved on the sheet: C010, C201, C203, C204, C416, C417, D501, D502, J001, J002, J003, J004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

Commit message: Added Precision Arduino 7400
Parts:
- removed R7: 10k, SparkFun-Passives:RESISTOR0603-RES
- added R6: 10k, KwanSystems:RP2EXB24V
- C201, C203, C204: device SparkFun:CAP0402-CAP -> SparkFun-Passives:CAP0603-CAP
- JP1, JP2, JP3, JP4: value STAND-OFF -> STANDOFF; device SparkFun:STAND-OFF -> KwanSystems:STANDOFF
- U401: value ATMEGA32U4TQFP -> ATMEGA32U4QFN2; device SparkFun-DigitalIC:ATMEGA32U4TQFP -> SparkFun-DigitalIC:ATMEGA32U4QFN2
Connections:
- net GND: now also JP1.P$1, JP2.P$1, JP3.P$1, JP4.P$1, R6A.1; no longer R7.1
- net HWB: now also R6A.2; no longer R7.2
- net MOSI: now also J003.4; no longer J003.2
- net RESET: now also J003.1, R6B.2; no longer J003.4
- net SCK: now also J003.5; no longer J003.1
- net VCC: now also J003.2, R6B.1; no longer J003.5
