File: 11Dof BMA180.sch (EAGLE design)
At the start: 20 parts, among them J401 M12PTH, U101 BMP180, U401 SN74LVC1G32, U501 L3G4200D, U601 BMA180, U801 5883

Commit message: RocketometerMPU sent to Laen
Parts:
- U401: DIGIKEY (none) -> 296-9847-2-ND
- U601: device SparkFun-Sensors:BMA180 -> KwanSystems:BMA180; DIGIKEY (none) -> $NOPART
Changed lines of the file:
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@@
 <attribute name="DIGIKEY" value="$NOPART"/>
 </part>
-<part name="U401" library="KwanSystems" deviceset="SN74LVC1G32" device=""/>
-<part name="U601" library="SparkFun-Sensors" deviceset="BMA180" device=""/>
+<part name="U401" library="KwanSystems" deviceset="SN74LVC1G32" device="">
+<attribute name="DIGIKEY" value="296-9847-2-ND"/>
+</part>
+<part name="U601" library="KwanSystems" deviceset="BMA180" device="">
+<attribute name="DIGIKEY" value="$NOPART"/>
+</part>
 </parts>
 <sheets>
@@
 <attribute name="DIGIKEY" x="116.84" y="228.6" size="1.778" layer="96" display="off"/>
 </instance>
-<instance part="U401" gate="G$1" x="195.58" y="200.66" rot="R180"/>
+<instance part="U401" gate="G$1" x="195.58" y="200.66" rot="R180">
+<attribute name="DIGIKEY" x="195.58" y="200.66" size="1.778" layer="96" display="off"/>
+</instance>
 <instance part="U401" gate="G$2" x="96.52" y="149.86" rot="R180"/>
-<instance part="U601" gate="G$1" x="50.8" y="254"/>
+<instance part="U601" gate="G$1" x="50.8" y="254">
+<attribute name="DIGIKEY" x="50.8" y="254" size="1.778" layer="96" display="off"/>
+</instance>
 </instances>
 <busses>
