File: 14DoF.brd (EAGLE design)
At the start: 30.5 x 12.7 mm, 24 parts, among them U101 BMP180, U601 MPU6050, U801 HMC5883L, U901 ADXL377, U902 AD7991

Commit message: 14DoF etc
Changed lines of the file:
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@@
 <text x="28.702" y="8.128" size="0.8128" layer="22" rot="MR0">Kwan Systems</text>
 <text x="9.398" y="2.794" size="0.8128" layer="21" rot="R90">IA</text>
-<text x="10.922" y="11.684" size="0.8128" layer="21">stkwans.blogspot.com</text>
+<text x="10.16" y="11.684" size="0.8128" layer="21">stkwans.blogspot.com</text>
 <rectangle x1="25.146" y1="4.318" x2="28.702" y2="7.874" layer="42" rot="R90"/>
 <rectangle x1="25.146" y1="7.112" x2="25.908" y2="7.874" layer="41"/>
@@
 </signal>
 </signals>
-<errors>
-</errors>
 </board>
 </drawing>

Commit message: Pushing back eagle changes
Parts:
- removed C907, C914: 100nF, SparkFun:0603-CAP
- added C921: 100nF, SparkFun-Passives:0603-CAP
- added C922: 4.7uF, SparkFun-Passives:0603-CAP
- added U920: MCP1525, KwanSystems:SOT-23-3
- moved C908 0.51 mm to (14.5, 10.2)
- moved C905 0.51 mm to (13.2, 10.2)
Connections:
- new net VREF: C922.1, U902.6, U920.2
- net GND: now also C921.2, C922.2, U920.3; no longer C907.2, C914.2
- net VCC: now also C921.1, U601.3, U920.1; no longer C907.1, C914.1
Routing:
- net VREF: track 0.00 -> 7.69 mm, vias 0 -> 1
- net VCC: track 60.0 -> 67.4 mm, vias 3 -> 4
Other:
- board text added: "31 May 2013"
- board text removed: "20 Nov 2012"
