File: KwanSystems/Precision/Precision Leonardo Charlieplex 2.0.brd (EAGLE design)
At the start: 76.2 x 76.2 mm, 152 parts, among them U201 3.3V, U401 ATMEGA32U4TQFP, Y401 16MHz

Commit message: Checked in Florida4 data
Parts:
- removed C001, C201: 1uF, SparkFun:0402-CAP
- removed C204: 100nF, SparkFun:0402-CAP
- removed C205: 4.7uF, SparkFun:0402-CAP
- removed U201: 3.3V, KwanSystems:SOT-23-5
- added C406, C501: 1uF, SparkFun-Passives:0603-CAP
- added C504: 100nF, SparkFun-Passives:0603-CAP
- added C505: 4.7uF, SparkFun-Passives:0603-CAP
- added J501: GP-2106, SparkFun:GP-2106
- added Q501, Q502: SSM6N58NU, KwanSystems:UDFN6
- added R501, R502: 10k, KwanSystems:CRA04
- added U501: 5319 1.8V, KwanSystems:SOT-23-5
- D408: value HOUR -> RED
- D422: value HOUR -> BLUE
- J001, J002: value (none) -> M04NOSILK; device SparkFun:1X04 -> KwanSystems:M04SIP
- J003, J004: value (none) -> M06NOSILK; device SparkFun:1X06 -> KwanSystems:M06SIP
- J405, J406: value (none) -> M08NOSILK; device SparkFun:1X08 -> KwanSystems:M08SIP
- JP1, JP2, JP3, JP4: value STAND-OFF -> STANDOFF; device SparkFun:STAND-OFF -> KwanSystems:STANDOFF
- moved J004 13.7 mm to (55.9, 44.5), turned to 270 degrees
Connections:
- removed net 3V3: C205.1, J004.2, J004.3, U201.5
- removed net N$17: C204.1, U201.4
- new net 1.8V: C505.1, J004.6, J501.VCC, Q501.2, Q501.5, Q502.2, Q502.5, R501.2, R501.4, R502.2, R502.4, U501.5
- new net 1PPS_I: J004.4, J501.1PPS, Q502.4, R502.5
- new net N$12: C504.1, U501.4
- new net ONOFF: Q502.6, R502.8, U401.26
- new net ONOFF_I: J004.3, J501.ONOFF, Q502.1, R502.7
- new net RX_I: J004.2, J501.RX, Q501.1, R501.5
- new net TX_O: J004.1, J501.TX, Q501.4, R501.7
- net AT_RX: now also Q501.3, R501.8; no longer J004.5
- net AT_TX: now also Q501.6, R501.6; no longer J004.6
- net GND: now also C406.1, C501.2, C504.2, C505.2, J004.5, J501.GND, JP1.P$1, JP2.P$1, JP3.P$1, JP4.P$1, U501.2; no longer C001.1, C201.2, C204.2, C205.2, J004.4, U201.2
- net N$1: now also C406.2; no longer C001.2
- net PPS: now also Q502.3, R502.6; no longer J004.1
- net VCC: now also C501.1, R501.1, R501.3, R502.1, R502.3, U501.1, U501.3; no longer C201.1, U201.1, U201.3
Routing:
- net 1.8V: track 0.00 -> 45.0 mm
- net VCC: track 86.7 -> 126.7 mm, vias 3 -> 2
- net ONOFF: track 0.00 -> 21.5 mm
- net 1PPS_I: track 0.00 -> 14.0 mm, vias 0 -> 1
- net RX_I: track 0.00 -> 13.9 mm, vias 0 -> 1
- net N$2: track 37.1 -> 49.1 mm, vias 2 -> 0
- net ONOFF_I: track 0.00 -> 11.4 mm, vias 0 -> 1
- net TX_O: track 0.00 -> 11.1 mm, vias 0 -> 1
- net AT_RX: track 30.6 -> 39.7 mm, vias 1 -> 2
- net SCK: track 20.1 -> 28.8 mm, vias 1 -> 0
- net 3V3: track 6.05 -> 0.00 mm
- net P03: track 20.4 -> 14.4 mm, vias 0 -> 2
- net PPS: track 21.1 -> 26.8 mm, vias 1 -> 4
- net RXLED: track 17.3 -> 12.9 mm
- net P01: track 28.5 -> 32.4 mm
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Other:
- board text added: "01 Apr 2014"
- board text added: "One board has controller, diodes clockwise"
- board text added: "One board has no controller, diodes counterclockwise"
- board text removed: "27 May 2013"
- board text removed: "3V3"
- board text removed: "BAT"
- board text removed: "One board has controller, diodes direct (pointing outwards)"
- board text removed: "One board has no controller, diodes reversed (pointing inwards)"
- board text removed: "PPS"
- board text removed: "R"
- board text removed: "RX"
- board text removed: "T"
- board text removed: "TX"
