File: KwanSystems/Precision/Precision Singleboard Leonardo Charlieplex.brd (EAGLE design)
At the start: 76.2 x 76.2 mm, 159 parts, among them Q501 SSM6N58NU, Q502 SSM6N58NU, U1 GP-2106, U201 1.8V, U401 ATMEGA328, U501 FT232RLSSOP, U602 ZF7, Y401 16MHz

Commit message: Checked in Florida4 data
Parts:
- removed C204: 1uF, SparkFun:0402-CAP
- removed C214: 100nF, SparkFun:0402-CAP
- removed C215: 4.7uF, SparkFun:0402-CAP
- removed C407, C408: 18pF, SparkFun:0603-CAP
- removed C418: 4.7uF, SparkFun:0603-CAP
- removed C502: 100nF, SparkFun:0603-CAP
- removed D501: BLUE, SparkFun:LED-0603
- removed D502: RED, SparkFun:LED-0603
- removed R13, R14, R606: 10k, KwanSystems:CRA04
- removed U1: GP-2106, SparkFun:GP-2106
- removed U201: 1.8V, KwanSystems:SOT-23-5
- removed U602: ZF7, KwanSystems:SC-70-6
- added C402: 4.7uF, SparkFun:0603-CAP
- added C406, C501: 1uF, SparkFun-Passives:0603-CAP
- added C416, C417: 18pF, SparkFun:0603-CAP
- added C504: 100nF, SparkFun-Passives:0603-CAP
- added C505: 4.7uF, SparkFun-Passives:0603-CAP
- added D200, D201, D202, D203, D204, D205, D206, D207, D208, D209, D210, D211, D212, D213, D214, D215, D216, D217, D218, D219, D220, D221, D222, D223, D224, D225, D226, D227, D228, D229, D230, D231, D232, D233, D234, D235, D236, D237, D238, D239, D240, D242, D243, D244, D245, D246, D247, D248, D249, D250, D251, D252, D253, D254, D255, D256, D257, D258, D259: SECOND, SparkFun-LED:LED-0603
- added D241: SECOND, SparkFun:LED-0603
- added D300, D301, D302, D303, D304, D305, D306, D307, D308, D309, D310, D311, D312, D313, D314, D315, D316, D317, D318, D319, D320, D321, D322, D323, D324, D325, D326, D327, D328, D329, D330, D331, D332, D333, D334, D335, D336, D337, D338, D339, D340, D341, D342, D343, D344, D345, D346, D347, D348, D349, D350, D351, D352, D353, D354, D355, D356, D357, D358, D359: THIRD, SparkFun-LED:LED-0603
- added D408: RED, SparkFun:LED-0603
- added D422: BLUE, SparkFun:LED-0603
- added J501: GP-2106, SparkFun:GP-2106
- added R403: 22, KwanSystems:CRA02
- added R413: 10k, KwanSystems:CRA02
- added R422: 680, KwanSystems:CRA02
- J004: device SparkFun-Connectors:1X05_NO_SILK -> SparkFun:1X06
- JP1, JP2, JP3, JP4: value STAND-OFF -> STANDOFF; device SparkFun:STAND-OFF -> KwanSystems:STANDOFF
- R501, R502: value 680 -> 10k; device SparkFun:0603-RES -> KwanSystems:CRA04
- U401: value ATMEGA328 -> ATMEGA32U4TQFP; device SparkFun:TQFP32-08 -> SparkFun-DigitalIC:SPARKFUN-DIGITALIC_TQFP44
- U501: value FT232RLSSOP -> 5319 1.8V; device SparkFun:SSOP28DB -> KwanSystems:SOT-23-5
- moved Q502 41.7 mm to (51.3, 36.8), turned to 270 degrees
- moved Q501 41.1 mm to (51.3, 39.4), turned to 270 degrees
- moved U501 22.2 mm to (59.7, 38.1)
- moved R502 21.0 mm to (51.3, 34.5), turned to 0 degrees
- moved R501 20.7 mm to (51.3, 41.7), turned to 180 degrees
- moved S429 18.1 mm to (25.1, 44.5)
- moved J004 13.7 mm to (55.9, 44.5), turned to 270 degrees
- moved Y401 13.1 mm to (29.2, 38.9), turned to 90 degrees
- moved C420 13.0 mm to (46.5, 40.6)
- moved U401 10.2 mm to (38.1, 38.1), turned to 270 degrees
- moved C010 0.25 mm to (35.8, 48.8)
Connections:
- removed net D12: J003.5, R606.8, U401.16, U602.6
- removed net GPS_TX: Q501.3, R13.1, U602.3
- removed net N$17: C214.1, U201.4
- removed net N$5: D501.C, R501.2
- removed net N$6: R501.1, U501.23
- removed net N$7: R502.1, U501.22
- removed net N$8: D502.C, R502.2
- removed net PPS_I: J004.1, Q502.4, R14.2, U1.1PPS
- removed net TX_I: J004.4
- removed net USB_TX: U501.1, U602.1
- new net 1PPS_I: J004.4, J501.1PPS, Q502.4, R502.2
- new net MISO: J003.5, U401.11
- new net MOSI: J003.6, U401.10
- new net N$1: C406.2, U401.6
- new net N$12: C504.1, U501.4
- new net N$2: R413.3, U401.33
- new net N$4: D408.A, R422.2
- new net RD+: R403.3, U401.4
- new net RD-: R403.4, U401.3
- new net RXLED: D408.C, U401.8
- new net SCK: J003.4, U401.9
- new net TXLED: D422.C, U401.22
- net 1.8V: now also C505.1, J004.6, J501.VCC, R501.6, R501.7, R502.6, R502.7, U501.5; no longer C215.1, J004.2, R13.6, R13.7, R14.6, R14.7, U1.VCC, U201.5
- net AREF: now also U401.42; no longer U401.20
- net AT_RX: now also Q501.3, R501.1, U401.20; no longer U401.30, U602.4
- net AT_TX: now also R501.4, U401.21; no longer R13.4, U401.31, U501.5
- net GND: now also C402.1, C406.1, C416.1, C417.1, C501.2, C504.2, C505.2, J004.5, J501.GND, JP1.P$1, JP2.P$1, JP3.P$1, JP4.P$1, R413.2, U401.15, U401.23, U401.35, U401.43, U501.2; no longer C204.2, C214.2, C215.2, C407.1, C408.1, C418.1, J004.3, U1.GND, U201.2, U401.21, U401.3, U501.18, U501.21, U501.25, U501.26, U501.7, U602.2
- net N$3: now also D422.A, R422.1; no longer C502.2, U501.2
- net ONOFF: now also R502.1, U401.26; no longer R14.1
- net ONOFF_I: now also J004.3, J501.ONOFF, R502.3; no longer R14.3, U1.ONOFF
- net P01: now also U401.12; no longer J003.6, U401.15
- net P02: now also U401.25; no longer U401.2
- net P03: now also U401.30; no longer U401.14
- net P04: now also U401.29; no longer U401.13
- net P05: now also U401.28; no longer U401.12
- net P06: now also U401.1; no longer U401.11
- net P07: now also U401.27; no longer U401.10
- net P08: now also U401.31; no longer U401.9
- net P09: now also U401.18; no longer U401.1
- net P10: now also U401.41; no longer U401.28
- net P11: now also U401.40; no longer U401.27
- net P12: now also U401.39; no longer U401.26
- net P13: now also U401.38; no longer U401.25
- net P14: now also U401.37; no longer U401.24
- net P15: now also U401.36; no longer U401.23
- net P16: now also U401.32; no longer J003.4, U401.17
- net PPS: now also R502.4, U401.19; no longer R14.4, U401.32
- net Q01: now also D200.A, D215.A, D229.A, D242.A, D254.A, D305.A, D315.A, D324.A, D332.A, D339.A, D345.A, D350.A, D354.A, D357.A, D359.A
- net Q02: now also D200.C, D201.A, D216.A, D230.A, D243.A, D255.A, D306.A, D316.A, D325.A, D333.A, D340.A, D346.A, D351.A, D355.A, D358.A
- net Q03: now also D201.C, D202.A, D215.C, D217.A, D231.A, D244.A, D256.A, D307.A, D317.A, D326.A, D334.A, D341.A, D347.A, D352.A, D356.A
- net Q04: now also D202.C, D203.A, D216.C, D218.A, D229.C, D232.A, D245.A, D257.A, D308.A, D318.A, D327.A, D335.A, D342.A, D348.A, D353.A
- net Q05: now also D203.C, D204.A, D217.C, D219.A, D230.C, D233.A, D242.C, D246.A, D258.A, D309.A, D319.A, D328.A, D336.A, D343.A, D349.A
- net Q06: now also D204.C, D205.A, D218.C, D220.A, D231.C, D234.A, D243.C, D247.A, D254.C, D259.A, D310.A, D320.A, D329.A, D337.A, D344.A
- net Q07: now also D205.C, D206.A, D219.C, D221.A, D232.C, D235.A, D244.C, D248.A, D255.C, D300.A, D305.C, D311.A, D321.A, D330.A, D338.A
- net Q08: now also D206.C, D207.A, D220.C, D222.A, D233.C, D236.A, D245.C, D249.A, D256.C, D301.A, D306.C, D312.A, D315.C, D322.A, D331.A
- net Q09: now also D207.C, D208.A, D221.C, D223.A, D234.C, D237.A, D246.C, D250.A, D257.C, D302.A, D307.C, D313.A, D316.C, D323.A, D324.C
- net Q10: now also D208.C, D209.A, D222.C, D224.A, D235.C, D238.A, D247.C, D251.A, D258.C, D303.A, D308.C, D314.A, D317.C, D325.C, D332.C
- net Q11: now also D209.C, D210.A, D223.C, D225.A, D236.C, D239.A, D248.C, D252.A, D259.C, D304.A, D309.C, D318.C, D326.C, D333.C, D339.C
- net Q12: now also D210.C, D211.A, D224.C, D226.A, D237.C, D240.A, D249.C, D253.A, D300.C, D310.C, D319.C, D327.C, D334.C, D340.C, D345.C
- net Q13: now also D211.C, D212.A, D225.C, D227.A, D238.C, D241.A, D250.C, D301.C, D311.C, D320.C, D328.C, D335.C, D341.C, D346.C, D350.C
- net Q14: now also D212.C, D213.A, D226.C, D228.A, D239.C, D251.C, D302.C, D312.C, D321.C, D329.C, D336.C, D342.C, D347.C, D351.C, D354.C
- net Q15: now also D213.C, D214.A, D227.C, D240.C, D252.C, D303.C, D313.C, D322.C, D330.C, D337.C, D343.C, D348.C, D352.C, D355.C, D357.C
- net Q16: now also D214.C, D228.C, D241.C, D253.C, D304.C, D314.C, D323.C, D331.C, D338.C, D344.C, D349.C, D353.C, D356.C, D358.C, D359.C
- net RESET: now also R413.1, U401.13; no longer C502.1, R606.5, U401.29
- net RX_I: now also J004.2, J501.RX, R501.2; no longer J004.5, R13.2, U1.RX
- net TX_O: now also J004.1, J501.TX, R501.3; no longer R13.3, U1.TX
- net USBD+: now also R403.2; no longer U501.15
- net USBD-: now also R403.1; no longer U501.16
- net VCC: now also C402.2, C501.1, R413.4, R422.3, R422.4, R501.5, R501.8, R502.5, R502.8, U401.14, U401.2, U401.24, U401.34, U401.44, U401.7, U501.1, U501.3; no longer C204.1, C418.2, D501.A, D502.A, R13.5, R13.8, R14.5, R14.8, R606.1, R606.4, U201.1, U201.3, U401.18, U401.4, U401.6, U501.20, U501.4, U602.5
- net XTAL1: now also C417.2, U401.17; no longer C407.2, U401.7
- net XTAL2: now also C416.2, U401.16; no longer C408.2, U401.8
Routing:
- net GND: track 0.00 -> 133.3 mm, vias 2 -> 4
- net D12: track 52.8 -> 0.00 mm, vias 3 -> 0
- net AT_RX: track 4.75 -> 47.9 mm, vias 0 -> 3
- net 1.8V: track 0.00 -> 40.7 mm, vias 0 -> 3
- net VCC: track 74.5 -> 114.2 mm, vias 3 -> 5
- net N$2: track 0.00 -> 39.1 mm, vias 0 -> 2
- net PPS: track 0.01 -> 30.4 mm, vias 0 -> 4
- net RESET: track 43.8 -> 14.6 mm, vias 2 -> 0
- net SCK: track 0.00 -> 27.8 mm
- net P06: track 8.01 -> 35.4 mm, vias 0 -> 2
- net P16: track 0.00 -> 26.9 mm, vias 0 -> 2
- net P11: track 0.02 -> 25.5 mm, vias 0 -> 2
- net P10: track 0.00 -> 25.4 mm, vias 0 -> 2
- net P12: track 0.00 -> 25.0 mm, vias 0 -> 2
- net ONOFF: track 0.00 -> 23.2 mm, vias 0 -> 2
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- added copper zone on layer 1, net GND
- added copper zone on layer 16, net GND
Other:
- board text added: "MOSI"
- board text added: "One board has controller, diodes clockwise"
- board text added: "One board has no controller, diodes counterclockwise"
- board text removed: "1V8"
- board text removed: "D11"
- board text removed: "One board has controller, diodes direct (pointing outwards)"
- board text removed: "One board has no controller, diodes reversed (pointing inwards)"
- board text removed: "PPS"
- board text removed: "RX"
- board text removed: "TX"

Commit message: More work on pure vector XR2 skin
Parts:
- removed J001: (no value), SparkFun:1X04
- removed J004: (no value), SparkFun:1X06
- removed J405, J406: (no value), SparkFun:1X08
- D100, D101, D102, D103, D104, D105, D106, D107, D108, D109, D110, D111, D112, D113, D114, D115, D116, D117, D118, D119, D120, D121, D122, D123, D124, D125, D126, D127, D128, D129, D130, D131, D132, D133, D134, D135, D136, D137, D138, D139, D140, D141, D142, D143, D144, D145, D146, D147, D148, D149, D150, D151, D152, D153, D154, D155, D156, D157, D158, D159: value HOUR -> MINUTE
- moved D359 653.2 mm to (34.3, 74.6), flipped to the bottom, turned to 264 degrees
- moved D358 644.3 mm to (30.5, 74.0), flipped to the bottom, turned to 258 degrees
- moved D357 635.5 mm to (26.7, 73.0), flipped to the bottom, turned to 252 degrees
- moved D356 626.7 mm to (23.2, 71.6), flipped to the bottom, turned to 246 degrees
- moved D355 618.1 mm to (19.7, 69.9), flipped to the bottom, turned to 240 degrees
- moved D354 609.6 mm to (16.5, 67.8), flipped to the bottom, turned to 234 degrees
- moved D353 601.3 mm to (13.5, 65.4), flipped to the bottom, turned to 228 degrees
- moved D352 593.3 mm to (10.8, 62.7), flipped to the bottom, turned to 222 degrees
- moved D351 585.5 mm to (8.41, 59.7), flipped to the bottom, turned to 216 degrees
- moved D350 578.0 mm to (6.32, 56.5), flipped to the bottom, turned to 210 degrees
- moved D349 570.9 mm to (4.57, 53.0), flipped to the bottom, turned to 204 degrees
- moved D348 564.2 mm to (3.20, 49.5), flipped to the bottom, turned to 198 degrees
- moved D347 557.8 mm to (2.21, 45.7), flipped to the bottom, turned to 192 degrees
- moved D346 551.8 mm to (1.60, 41.9), flipped to the bottom, turned to 186 degrees
- moved D345 546.3 mm to (1.40, 38.1), flipped to the bottom, turned to 180 degrees
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Connections:
- net 1.8V: no longer J004.6
- net 1PPS_I: no longer J004.4
- net GND: no longer J001.4, J004.5
- net ONOFF_I: no longer J004.3
- net Q01: no longer J406.1
- net Q02: no longer J406.2
- net Q03: no longer J406.3
- net Q04: no longer J406.4
- net Q05: no longer J406.5
- net Q06: no longer J406.6
- net Q07: no longer J406.7
- net Q08: no longer J406.8
- net Q09: no longer J405.1
- net Q10: no longer J405.2
- net Q11: no longer J405.3
- net Q12: no longer J405.4
- net Q13: no longer J405.5
- net Q14: no longer J405.6
- net Q15: no longer J405.7
- net Q16: no longer J405.8
- net RX_I: no longer J004.2
- net TX_O: no longer J004.1
- net USBD+: no longer J001.1
- net USBD-: no longer J001.2
- net VCC: no longer J001.3
Routing:
- net GND: track 133.3 -> 0.00 mm, vias 4 -> 7
- net AT_TX: track 33.4 -> 49.2 mm, vias 4 -> 3
- net AT_RX: track 47.9 -> 32.9 mm
- net ONOFF: track 23.2 -> 34.3 mm, vias 2 -> 4
- net ONOFF_I: track 17.9 -> 8.62 mm
- net 1PPS_I: track 17.6 -> 10.2 mm, vias 1 -> 2
- net Q10: track 303.3 -> 309.8 mm, vias 21 -> 22
- net Q02: track 265.4 -> 271.7 mm, vias 19 -> 20
- net Q07: track 284.1 -> 289.5 mm, vias 21 -> 22
- net Q08: track 288.6 -> 293.9 mm, vias 21 -> 22
- net TX_O: track 17.4 -> 12.1 mm
- net RX_I: track 15.6 -> 10.3 mm, vias 1 -> 2
- net PPS: track 30.4 -> 35.4 mm
- net P08: track 17.4 -> 22.3 mm
- net Q09: track 296.7 -> 301.2 mm, vias 21 -> 22
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Other:
- board text added: "01 Apr 2014"
- board text removed: "27 May 2013"
- board text removed: "One board has controller, diodes clockwise"
- board text removed: "One board has no controller, diodes counterclockwise"

Commit message: Shuffled several documents
Routing:
- net Q04: track 269.6 -> 271.0 mm
- net Q10: track 309.8 -> 310.6 mm
- net Q12: track 304.9 -> 305.6 mm
