File: KwanSystems/Arisa/Engine Room v3.brd (EAGLE design)
At the start: 72.4 x 35.6 mm, 28 parts, among them Q201 IRF6718, Q202 IRF6718, U101 PC847, U201 L298

Commit message: More work on Yukari, replaced transistor with my own library, which includes SC70 package
Parts:
- Q201, Q202: value IRF6718 -> MOSFET_NCHANNELIRF6718
Changed lines of the file:
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@@
 <element name="C1" library="SparkFun" package="0402-CAP" value="" x="56.642" y="22.606"/>
 <element name="C2" library="SparkFun" package="0402-CAP" value="" x="57.15" y="25.654" rot="R180"/>
-<element name="Q201" library="KwanSystems" package="DIRECTFET_L6" value="IRF6718" x="57.15" y="31.75"/>
-<element name="Q202" library="KwanSystems" package="DIRECTFET_L6" value="IRF6718" x="57.15" y="3.81"/>
+<element name="Q201" library="KwanSystems" package="DIRECTFET_L6" value="MOSFET_NCHANNELIRF6718" x="57.15" y="31.75"/>
+<element name="Q202" library="KwanSystems" package="DIRECTFET_L6" value="MOSFET_NCHANNELIRF6718" x="57.15" y="3.81"/>
 </elements>
 <signals>
