File: KwanSystems/Arisa/Engine Room.sch (EAGLE design)
At the start: 25 parts, among them Q201 IRF6718, Q202 IRF6718, U101 PC847, U201 LMD1820X

Commit message: More work on Yukari, replaced transistor with my own library, which includes SC70 package
Parts:
- Q201, Q202: value IRF6718 -> MOSFET_NCHANNELIRF6718; device KwanSystems:IRF6718 -> KwanSystems:MOSFET_NCHANNELIRF6718
Changed lines of the file:
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@@
 <part name="M1" library="SparkFun" deviceset="M02" device="PTH4"/>
 <part name="M2" library="SparkFun" deviceset="M02" device="PTH4"/>
-<part name="Q201" library="KwanSystems" deviceset="IRF6718" device=""/>
-<part name="Q202" library="KwanSystems" deviceset="IRF6718" device=""/>
+<part name="Q201" library="KwanSystems" deviceset="MOSFET_NCHANNEL" device="IRF6718"/>
+<part name="Q202" library="KwanSystems" deviceset="MOSFET_NCHANNEL" device="IRF6718"/>
 </parts>
 <sheets>
