File: KwanSystems/Arisa/LPC2148 Engine Room.brd (EAGLE design)
At the start: 66 x 45.7 mm, 72 parts, among them J004 USB_MICROB_JSTGCT, J301 JST 2mm, J401 M07, J701 MICROSD-SOCKET, Q050 PMOS, Q201 IRF6718, Q202 IRF6718, U003 LPC2148, U004 5319, U101 BMP180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

Commit message: More work on Yukari, replaced transistor with my own library, which includes SC70 package
Parts:
- Q201, Q202: value IRF6718 -> MOSFET_NCHANNELIRF6718
Changed lines of the file:
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@@
 <element name="R201" library="KwanSystems" package="CRA04" value="1k" x="35.56" y="10.922" rot="R180"/>
 <element name="R203" library="KwanSystems" package="CRA04" value="220" x="24.765" y="36.703" rot="R180"/>
-<element name="Q201" library="KwanSystems" package="DIRECTFET_L6" value="IRF6718" x="50.8" y="41.91">
+<element name="Q201" library="KwanSystems" package="DIRECTFET_L6" value="MOSFET_NCHANNELIRF6718" x="50.8" y="41.91">
 <attribute name="LOGO_3D50" value="NOLOGO" x="50.8" y="41.91" size="1.778" layer="21" display="off"/>
 </element>
-<element name="Q202" library="KwanSystems" package="DIRECTFET_L6" value="IRF6718" x="50.8" y="3.81">
+<element name="Q202" library="KwanSystems" package="DIRECTFET_L6" value="MOSFET_NCHANNELIRF6718" x="50.8" y="3.81">
 <attribute name="LOGO_3D50" value="NOLOGO" x="50.8" y="3.81" size="1.778" layer="21" display="off"/>
 </element>
@@
 </signal>
 </signals>
-<errors>
-</errors>
 </board>
 </drawing>
