File: KwanSystems/Arisa/Engine Room Power Half.sch (EAGLE design)
At the start: 48 parts, among them J001 USB_MICROB_JSTGCT, J002 M15, J003 M15, Q201 MOSFET_NCHANNELIRF6718, Q202 MOSFET_NCHANNELIRF6718, U001 FT232RLSSOP, U201 L298, U202 PC847, U203 MC74VHC1G04, U204 UA78M05, U401 ATMEGA328P

Commit message: Reorganized docs for ARM. Added engine rooms with AD magnetic couplers instead of optocouplers.
Parts:
- removed C002, C404, C406, C418, C420: 100nF, SparkFun:CAP0402-CAP
- removed C201: 1uF, SparkFun:CAP0402-CAP
- removed C203: 4.7uF, SparkFun:CAP0402-CAP
- removed C407, C408: 18pF, SparkFun:CAP0402-CAP
- removed D003: MSS1P6, KwanSystems:MSS1P6
- removed D022: BLUE, SparkFun-LED:LED0603
- removed D023: RED, SparkFun-LED:LED0603
- removed D401: GREEN, SparkFun-LED:LED0603
- removed D402: YELLOW, SparkFun-LED:LED0603
- removed J001: USB_MICROB_JSTGCT, KwanSystems:USB_MICROB_JSTGCT
- removed J002, J003: M15, SparkFun-Connectors:M15
- removed JP3, JP4: (no value), SparkFun-Connectors:M03PTH
- removed R001: 680, KwanSystems:RP404
- removed R201: 1k, KwanSystems:RP404
- removed R203: 220, KwanSystems:RP404
- removed R429: 10k, SparkFun-Passives:RESISTOR0402-RES
- removed S429: B3U-1000P, KwanSystems:B3U-1000P
- removed U001: FT232RLSSOP, SparkFun-DigitalIC:FT232RLSSOP
- removed U002: (no value), KwanSystems:MAX8881
- removed U202: PC847, optocoupler:PC847
- removed U401: ATMEGA328P, SparkFun-DigitalIC:ATMEGA168
- added C1, C2: 100nF, SparkFun:CAP0402-CAP
- added C3, C4: 10uF, SparkFun-Passives:CAP1206
- added U$5: ADUM3221, KwanSystems:ADUM3221
- C214: device SparkFun:CAP0402-CAP -> SparkFun-Passives:CAP1206
- U$3: value (none) -> ADUM3221; device KwanSystems:CX2520 -> KwanSystems:ADUM3221
- U204: device MySMD:UA78M05 -> KwanSystems:UA78M05
Connections:
- removed net 3V3: J003.2, U001.3V3OUT
- removed net A0: J003.4, U401.PC0(ADC0)
- removed net A1: J003.5, U401.PC1(ADC1)
- removed net A2: J003.6, U401.PC2(ADC2)
- removed net A3: J003.7, U401.PC3(ADC3)
- removed net A4: J003.8, U401.PC4(ADC4/SDA)
- removed net A5: J003.9, U401.PC5(ADC5/SCL)
- removed net A6: J003.10, U401.ADC6
- removed net A7: J003.11, U401.ADC7
- removed net AREF: C420.1, J003.3, U401.AREF
- removed net D0: J002.1, U001.TXD, U401.PD0(RXD)
- removed net D1: J002.2, U001.RXD, U401.PD1(TXD)
- removed net D10: J002.13, U401.PB2(SS/OC1B)
- removed net D11: J002.14, JP4.2, U401.PB3(MOSI/OC2)
- removed net D12: J002.15, JP3.1, U401.PB4(MISO)
- removed net D13: J003.1, JP3.2, R001D.2, U401.PB5(SCK)
- removed net D2: J002.5, U401.PD2(INT0)
- removed net D3: J002.6, R203D.1, U401.PD3(INT1)
- removed net D3_ISO: R203D.2, U202D.C
- removed net D4: J002.7, U401.PD4(XCK/T0)
- removed net D5: J002.8, R203B.1, U401.PD5(T1)
- removed net D5_ISO: R203B.2, U202B.C
- removed net D6: J002.9, R203C.1, U401.PD6(AIN0)
- removed net D6_ISO: R203C.2, U202C.C
- removed net D7: J002.10, U401.PD7(AIN1)
- removed net D8: J002.11, U401.PB0(ICP)
- removed net D9: J002.12, R203A.1, U401.PB1(OC1A)
- removed net D9_ISO: R203A.2, U202A.C
- removed net DTR#: C002.2, U001.DTR
- removed net N$10: C219.1, R202.2, U201.VLS, U203PWR.VCC, U204.OUT
- removed net N$11: D023.A, R001A.1
- removed net N$28: R201C.1, U201.ENA, U201.ENB, U202C.EMIT
- removed net N$3: C407.2, U$3.1, U401.PB6(XTAL1/TOSC1)
- removed net N$35: Q201.G, R201A.1, U202A.EMIT
- removed net N$36: Q202.G, R201D.1, U202D.EMIT
- removed net N$37: R201B.1, U201.IN2, U201.IN3, U202B.EMIT, U203A.A
- removed net N$4: C408.2, U$3.2, U401.PB7(XTAL2/TOSC2)
- removed net N$5: J001.D+, U001.USBDP
- removed net N$6: J001.D-, U001.USBDM
- removed net N$7: D401.A, R001C.1
- removed net N$8: D402.A, R001D.1
- removed net N$9: D022.A, R001B.1
- removed net RESET: C002.1, J002.3, J003.13, JP3.3, R429.2, S429.2, U401.PC6(/RESET)
- removed net RXLED1: D022.C, U001.RXLED
- removed net TXLED1: D023.C, U001.TXLED
- removed net VBUS: D003.A, J001.VBUS
- removed net VIN: C201.1, J003.15, U002.IN, U002.SHDN#
- new net MT_DIR: U$5A.IN
- new net MT_DIR_G: U$5A.OUT, U201.IN2, U201.IN3, U203A.A
- new net PVCC: C219.1, C4.1, R202.2, U$5OUTP.VCC, U201.VLS, U203PWR.VCC, U204.VOUT
- new net PWMB: U$5B.IN
- new net PWMB_G: U$5B.OUT, U201.ENA, U201.ENB
- new net PWMG: U$3B.IN
- new net PWMG_G: Q202.G, U$3B.OUT
- new net PWMR: U$3A.IN
- new net PWMR_G: Q201.G, U$3A.OUT
- net GND: now also C1.2, C2.2, U$3INP.GND, U$5INP.GND; no longer C201.2, C203.2, C404.2, C406.2, C407.1, C408.1, C418.2, C420.2, D401.C, D402.C, J001.GND, J002.4, J003.14, JP4.1, S429.1, U$3.GND, U001.AGND, U001.GND18, U001.GND21, U001.GND7, U001.TEST, U002.GND, U401.AGND, U401.GND@1, U401.GND@2
- net PGND: now also C3.2, C4.2, U$3OUTP.GND, U$5OUTP.GND, U204.GND; no longer R201A.2, R201B.2, R201C.2, R201D.2, U204.GND1, U204.GND2
- net VCC: now also C1.1, C2.1, U$3INP.VCC, U$5INP.VCC; no longer C203.1, C404.1, C406.1, C418.1, D003.K, J003.12, JP4.3, R001A.2, R001B.2, R001C.2, R429.1, U001.VCC, U001.VCCIO, U002.FB, U002.OUT, U202A.A, U202B.A, U202C.A, U202D.A, U401.AVCC, U401.VCC@1, U401.VCC@2
- net VDD: now also C3.1, U$3OUTP.VCC, U204.VCC; no longer U202A.COL, U202B.COL, U202C.COL, U202D.COL, U204.IN
Other:
- note added: "H H H Brake"
- note added: "H L H Reverse"
- note added: "IN1 IN2 ENA Function"
- note added: "In1 needs to be in parallel with In4, and In2 with In3."
- note added: "L H H Forward"
- note added: "L L H Brake"
- note added: "L298 is a dual H-bridge, used in parallel here. Needs"
- note added: "Likewise Out1 and Out4. We probably don't need this much current,"
- note added: "M2 PWM"
- note added: "We put the PWM signal on ENA and run DIR through an inverter"
- note added: "X X L Free-wheel"
- note added: "a 5V regulator for logic power, since it can handle"
- note added: "but the other channel would be idle otherwise."
- note added: "logic side. Isolator high-side is powered off this as well."
- note added: "the motor free-wheels rather than braking when the PWM signal is low."
- note added: "to get complementary signals to apply to IN1 and IN2. This way,"
- note added: "up to 50V on the power side but not more than 7V on the"
- note removed: "Arduino Nano v3.0"
- note removed: "Controller circuit below derived from"
- note removed: "Copyright 2009 under the Creative Commons Attribution Share-Alike 2.5 License"
- note removed: "gravitech.us"
- note removed: "http://creativecommons.org/license/by-sa/2.5/"
- moved on the sheet: C214, D202, M1, M2, Q202
