File: KwanSystems/Arisa/LPC2148 Engine Room ADUM.sch (EAGLE design)
At the start: 48 parts, among them J001 USB_MICROB_JSTGCT, J002 M15, J003 M15, Q201 MOSFET_NCHANNELIRF6718, Q202 MOSFET_NCHANNELIRF6718, U001 FT232RLSSOP, U201 L298, U202 PC847, U203 MC74VHC1G04, U204 UA78M05, U401 ATMEGA328P

Commit message: Reorganized docs for ARM. Added engine rooms with AD magnetic couplers instead of optocouplers.
Parts:
- removed C002, C404, C406, C418, C420: 100nF, SparkFun:CAP0402-CAP
- removed C201: 1uF, SparkFun:CAP0402-CAP
- removed C203: 4.7uF, SparkFun:CAP0402-CAP
- removed C407, C408: 18pF, SparkFun:CAP0402-CAP
- removed D003: MSS1P6, KwanSystems:MSS1P6
- removed D022: BLUE, SparkFun-LED:LED0603
- removed D023: RED, SparkFun-LED:LED0603
- removed D401: GREEN, SparkFun-LED:LED0603
- removed D402: YELLOW, SparkFun-LED:LED0603
- removed J001: USB_MICROB_JSTGCT, KwanSystems:USB_MICROB_JSTGCT
- removed J002, J003: M15, SparkFun-Connectors:M15
- removed JP3, JP4: (no value), SparkFun-Connectors:M03PTH
- removed R001: 680, KwanSystems:RP404
- removed R201: 1k, KwanSystems:RP404
- removed R203: 220, KwanSystems:RP404
- removed R429: 10k, SparkFun-Passives:RESISTOR0402-RES
- removed S429: B3U-1000P, KwanSystems:B3U-1000P
- removed U001: FT232RLSSOP, SparkFun-DigitalIC:FT232RLSSOP
- removed U002: (no value), KwanSystems:MAX8881
- removed U202: PC847, optocoupler:PC847
- removed U401: ATMEGA328P, SparkFun-DigitalIC:ATMEGA168
- added C001, C101, C443, C449, C610, C613: 100nF, SparkFun:CAP0402-CAP
- added C003, C301, C302: 4.7uF, SparkFun:CAP0402-CAP
- added C023: 22pF, KwanSystems:CKCM25
- added C204, C423, C451, C463: 1uF, SparkFun:CAP0402-CAP
- added C461, C462: 33pF, SparkFun:CAP0402-CAP
- added C620: 2.2nF, SparkFun:CAP0402-CAP
- added C901: 10uF, SparkFun:CAP0603-CAP
- added C906: 100nF, SparkFun-Passives:CAP0402-CAP
- added D001: SMLP36RGB2W(R), KwanSystems:SMLP36RGB2W(R)
- added D050: BLUE, SparkFun:LED0603
- added D301: YELLOW, SparkFun:LED0603
- added D302: DCC, KwanSystems:PMEG2005CT
- added J004: USB_MICROB_JSTGCT, KwanSystems:USB_MICROB_JSTGCT
- added J301: JST 2mm, SparkFun:M02-JST-2MM-SMT
- added J401: M07, SparkFun-Connectors:M081X08
- added J701: MICROSD-SOCKET, KwanSystems:MICROSD-SOCKET
- added Q050: PMOS, SparkFun:MOSFET-PCHANNELSMD
- added R011: 100k, SparkFun:RESISTOR0402-RES
- added R015: 10k, KwanSystems:RP2EXB24V
- added R023: 33, KwanSystems:RP2EXB24V
- added R053, R402: 1.5k, KwanSystems:RP404
- added R301: 10k, SparkFun:RESISTOR0402-RES
- added R302: 1M, KwanSystems:RP2EXB24V
- added R401: 10k, KwanSystems:RP404
- added S201: AYZ0202, KwanSystems:AYZ0202
- added S457, S458: B3U-1100P, KwanSystems:B3U-1100P
- added S457A: SOLDERJUMPERNO, SparkFun-Passives:SOLDERJUMPERNO
- added U$5: ADUM3221, KwanSystems:ADUM3221
- added U003: LPC2148, SparkFun:LPC213X
- added U004: 5319, KwanSystems:MIC5319D5
- added U101: BMP180, KwanSystems:BMP180
- added U301: 73831, SparkFun:MCP73831
- added U601: MPU9150, KwanSystems:MPU9150
- added U902: ADXL375, KwanSystems:ADXL375
- added Y401: 12MHz, KwanSystems:CX2520
- U$3: value (none) -> ADUM3221; device KwanSystems:CX2520 -> KwanSystems:ADUM3221
- U204: device MySMD:UA78M05 -> KwanSystems:UA78M05
Connections:
- removed net 3V3: J003.2, U001.3V3OUT
- removed net A0: J003.4, U401.PC0(ADC0)
- removed net A1: J003.5, U401.PC1(ADC1)
- removed net A2: J003.6, U401.PC2(ADC2)
- removed net A3: J003.7, U401.PC3(ADC3)
- removed net A4: J003.8, U401.PC4(ADC4/SDA)
- removed net A5: J003.9, U401.PC5(ADC5/SCL)
- removed net A6: J003.10, U401.ADC6
- removed net A7: J003.11, U401.ADC7
- removed net AREF: C420.1, J003.3, U401.AREF
- removed net D0: J002.1, U001.TXD, U401.PD0(RXD)
- removed net D1: J002.2, U001.RXD, U401.PD1(TXD)
- removed net D10: J002.13, U401.PB2(SS/OC1B)
- removed net D11: J002.14, JP4.2, U401.PB3(MOSI/OC2)
- removed net D12: J002.15, JP3.1, U401.PB4(MISO)
- removed net D13: J003.1, JP3.2, R001D.2, U401.PB5(SCK)
- removed net D2: J002.5, U401.PD2(INT0)
- removed net D3: J002.6, R203D.1, U401.PD3(INT1)
- removed net D3_ISO: R203D.2, U202D.C
- removed net D4: J002.7, U401.PD4(XCK/T0)
- removed net D5: J002.8, R203B.1, U401.PD5(T1)
- removed net D5_ISO: R203B.2, U202B.C
- removed net D6: J002.9, R203C.1, U401.PD6(AIN0)
- removed net D6_ISO: R203C.2, U202C.C
- removed net D7: J002.10, U401.PD7(AIN1)
- removed net D8: J002.11, U401.PB0(ICP)
- removed net D9: J002.12, R203A.1, U401.PB1(OC1A)
- removed net D9_ISO: R203A.2, U202A.C
- removed net DTR#: C002.2, U001.DTR
- removed net N$10: C219.1, R202.2, U201.VLS, U203PWR.VCC, U204.OUT
- removed net N$11: D023.A, R001A.1
- removed net N$28: R201C.1, U201.ENA, U201.ENB, U202C.EMIT
- removed net N$3: C407.2, U$3.1, U401.PB6(XTAL1/TOSC1)
- removed net N$35: Q201.G, R201A.1, U202A.EMIT
- removed net N$36: Q202.G, R201D.1, U202D.EMIT
- removed net N$37: R201B.1, U201.IN2, U201.IN3, U202B.EMIT, U203A.A
- removed net N$4: C408.2, U$3.2, U401.PB7(XTAL2/TOSC2)
- removed net N$5: J001.D+, U001.USBDP
- removed net N$6: J001.D-, U001.USBDM
- removed net N$7: D401.A, R001C.1
- removed net N$8: D402.A, R001D.1
- removed net N$9: D022.A, R001B.1
- removed net RXLED1: D022.C, U001.RXLED
- removed net TXLED1: D023.C, U001.TXLED
- new net ACCINT: U003.(CAP1.2/SCK1/MAT1.2)P0.17, U601.INT
- new net BATLVL: R302A.2, R302B.2, U003.(AD0.3/EINT3/CAP0.0)P0.30
- new net BSL: J401.5, R401A.1, U003.(DCD1/EINT1/SDA1)P0.14
- new net CONN_D+: J004.D+, R023B.1, R053B.2
- new net CONN_D-: J004.D-, R023A.1
- new net CS0: J701./CS, U003.(RI1/EINT2/AD1.5)P0.15
- new net EN: S201B.P$3, U004.EN
- new net MISO0: J701.DO, U003.(MISO0/MAT0.1/A0.7)P0.5
- new net MOSI0: J701.DI, U003.(MOSI0/CAP0.2/AD1.0)P0.6
- new net MT_DIR: U$5A.IN, U003.(RTS1/CAP1.0/AD1.2)P0.10
- new net MT_DIR_G: U$5A.OUT, U201.IN2, U201.IN3, U203A.A
- new net N$12: C620.2, U601.CPOUT
- new net N$13: C610.1, U601.REGOUT
- new net N$14: S457A.2, S457S.1
- new net N$15: R301.2, U301.PROG
- new net N$16: D050.C, R053A.2
- new net N$17: C001.1, U004.BYP
- new net N$18: D301.A, R053D.1
- new net N$19: D301.C, U301.STAT
- new net N$20: D050.A, Q050.D, R053B.1
- new net PVCC: C219.1, R202.2, U$5OUTP.VCC, U201.VLS, U203PWR.VCC, U204.VOUT
- new net PWMB: R402A.2, U$5B.IN, U003.(SSEL0/PWM2/EINT2)P0.7
- new net PWMB_G: U$5B.OUT, U201.ENA, U201.ENB
- new net PWMG: R402D.2, U$3B.IN, U003.(RXD1/PWM6/EINT3)P0.9
- new net PWMG_G: Q202.G, U$3B.OUT
- new net PWMR: R402B.2, U$3A.IN, U003.(TXD1/PWM4/A1.1)P0.8
- new net PWMR_G: Q201.G, U$3A.OUT
- new net QWMB: D001B.C, R402A.1
- new net QWMG: D001G.C, R402D.1
- new net QWMR: D001R.C, R402B.1
- new net RX0: J401.3, U003.(RXD0/PWM3/EINT0)P0.1
- new net SCK0: J701.SCK, U003.(SCK0/CAP0.1/AD0.6)P0.4
- new net SCL0: J401.6, R401D.1, U003.(SCL0/CAP0.0)P0.2, U101.SCL, U601.SCL, U902.SCL/SCK
- new net SDA0: J401.7, R401C.1, U003.(SDA0/MAT0.0/EINT1)P0.3, U101.SDA, U601.SDA, U902.SDA/SDI/SDIO
- new net TX0: J401.2, U003.(TXD0/PWM1)P0.0
- new net USBD+: C023B.1, R023B.2, U003.(AD0.5)P0.26
- new net USBD-: C023A.1, R023A.2, U003.(AD0.0/CAP0.1/MAT0.1)P0.27
- new net USB_ON: R015B.1, S458S.2, U003.P0.23
- new net USB_SOFTCONNECT: Q050.G, R015A.2, U003.P0.31
- new net VLIPO: C301.1, C449.2, D302.A2, J301.2, R302B.1, U003.VBAT, U301.VBAT
- new net XTAL1: C462.2, U003.XTAL1, Y401.1
- new net XTAL2: C461.2, U003.XTAL2, Y401.2
- net GND: now also C001.2, C003.2, C023A.2, C023B.2, C101.2, C204.2, C301.2, C302.2, C423.2, C443.2, C449.1, C451.2, C461.1, C462.1, C463.2, C610.2, C613.1, C620.1, C901.2, C906.2, J004.GND, J301.1, J401.4, J701.GND, J701.SHIELD, R011.1, R053A.1, R301.1, R302A.1, S201B.P$1, S457G.1, S457S.2, S458G.1, S458S.1, U$3INP.GND, U$5INP.GND, U003.RTXC1, U003.VSS, U003.VSS@1, U003.VSS@2, U003.VSS@3, U003.VSS@4, U003.VSSA, U004.GND, U101.GND, U301.VSS, U601.AD0, U601.CLKIN, U601.FSYNC, U601.GND, U902.GND, U902.SDO/AA, Y401.GND; no longer C201.2, C203.2, C404.2, C406.2, C407.1, C408.1, C418.2, C420.2, D401.C, D402.C, J001.GND, J002.4, J003.14, JP4.1, S429.1, U$3.GND, U001.AGND, U001.GND18, U001.GND21, U001.GND7, U001.TEST, U002.GND, U401.AGND, U401.GND@1, U401.GND@2
- net PGND: now also U$3OUTP.GND, U$5OUTP.GND, U204.GND; no longer R201A.2, R201B.2, R201C.2, R201D.2, U204.GND1, U204.GND2
- net RESET: now also R401B.1, S457A.1, U003.RESET; no longer C002.1, J002.3, J003.13, JP3.3, R429.2, S429.2, U401.PC6(/RESET)
- net VBUS: now also C302.1, D302.A1, J004.VBUS, J401.1, R011.2, R015B.2, R053D.2, U301.VIN; no longer D003.A, J001.VBUS
- net VCC: now also C003.1, C101.1, C423.1, C443.1, C451.1, C463.1, C613.2, C901.1, C906.1, D001B.A, D001G.A, D001R.A, J401.8, J701.VCC, Q050.S, R015A.1, R401A.2, R401B.2, R401C.2, R401D.2, U$3INP.VCC, U$5INP.VCC, U003.VDD3-1, U003.VDD3-2, U003.VDD3-3, U003.VDDA3, U003.VREF, U004.VOUT, U101.VDD, U101.VDDIO, U601.VDD, U601.VLOGIC, U902.CS, U902.VDDIO, U902.VS; no longer C203.1, C404.1, C406.1, C418.1, D003.K, J003.12, JP4.3, R001A.2, R001B.2, R001C.2, R429.1, U001.VCC, U001.VCCIO, U002.FB, U002.OUT, U202A.A, U202B.A, U202C.A, U202D.A, U401.AVCC, U401.VCC@1, U401.VCC@2
- net VDD: now also U$3OUTP.VCC, U204.VCC; no longer U202A.COL, U202B.COL, U202C.COL, U202D.COL, U204.IN
- net VIN: now also C204.1, D302.K, S201B.P$2, U004.VIN; no longer C201.1, J003.15, U002.IN, U002.SHDN#
Other:
- note added: "10MHz-15MHz 10pF <300 18pF"
- note added: "10MHz-15MHz 20pF <220 38pF"
- note added: "10MHz-15MHz 30pF <140 58pF"
- note added: "32kiHz 11pF <100k 18pF"
- note added: "32kiHz 13pF <100k 22pF"
- note added: "32kiHz 15pF <100k 27pF"
- note added: "Abracon ABS06 32kiHz - 12.5pf Cl <90k Rs 20ppm"
- note added: "D"
- note added: "Freq Cl Rs Cx1,Cx2"
- note added: "G"
- note added: "H H H Brake"
- note added: "H L H Reverse"
- note added: "IN1 IN2 ENA Function"
- note added: "In1 needs to be in parallel with In4, and In2 with In3."
- note added: "L H H Forward"
- note added: "L L H Brake"
- note added: "L298 is a dual H-bridge, used in parallel here. Needs"
- note added: "Likewise Out1 and Out4. We probably don't need this much current,"
- note added: "M2 PWM"
- note added: "OR Y401/C461/C462"
- note added: "Place either Y403/C404"
- note added: "S"
- note added: "Section 0 - USB interface"
- note added: "Section 1 - Baro/Temp sensor"
- note added: "Section 2 - Regulator"
- note added: "Section 3 - Charging circuit"
- note added: "Section 4 - Controller"
- note added: "Section 7 - MicroSD"
- note added: "Section 9 - Digital HighAcc"
- note added: "TXC inc 8Z 12MHz - 18pf Cl <100 Rs 30ppm/30ppm"
- note added: "We put the PWM signal on ENA and run DIR through an inverter"
- note added: "X X L Free-wheel"
- note added: "a 5V regulator for logic power, since it can handle"
- note added: "at 12.5pF, exact Cx1 is 21pF, 22pF is closest E12"
- note added: "at 18pF, exact Cx1 is 34pF, 33pF is closest E12"
- note added: "but not both groups"
- note added: "but the other channel would be idle otherwise."
- note added: "logic side. Isolator high-side is powered off this as well."
- note added: "the motor free-wheels rather than braking when the PWM signal is low."
- note added: "to get complementary signals to apply to IN1 and IN2. This way,"
- note added: "up to 50V on the power side but not more than 7V on the"
- note removed: "Arduino Nano v3.0"
- note removed: "Controller circuit below derived from"
- note removed: "Copyright 2009 under the Creative Commons Attribution Share-Alike 2.5 License"
- note removed: "gravitech.us"
- note removed: "http://creativecommons.org/license/by-sa/2.5/"
- moved on the sheet: D202, M1, M2, Q202
