File: KwanSystems/Yukari/Yukari.brd (EAGLE design)
At the start: 55.9 x 22.9 mm, 62 parts, among them J001 USB_MICROB_JSTGCT, J301 JST 2mm, J401 M07, J501 GP-2106, J701 MICROSD-SOCKET, Q050 PMOS, U101 BMP180, U201 5319 3.3V, U301 73831, U401 LPC2148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

Commit message: Branched Rocketometer off into Yukari
Parts:
- removed C301: 4.7uF, SparkFun:0402-CAP
- removed D301: YELLOW, SparkFun:LED-0603
- removed D302: DCC, KwanSystems:SOT-23-3
- removed J301: JST 2mm, SparkFun:JST-2-SMD
- removed R301: 10k, SparkFun:0402-RES
- removed S201: AYZ0202, KwanSystems:AYZ0202
- removed S458: B3U-1100P, KwanSystems:B3U-1100P
- removed U301: 73831, SparkFun:SOT23-5
- D402: value DIODE_SCHOTTKY -> DIODE_COMMON_CATHODEBAT30C; device KwanSystems:D0603 -> KwanSystems:SC-70-3
- J401: value M07 -> (none); device SparkFun-Connectors:1X11 -> SparkFun-Connectors:1X15
- R053: device KwanSystems:CRA04 -> KwanSystems:CRA02
- moved J401 10.2 mm to (47.0, 21.6)
- moved C302 8.85 mm to (48.3, 14.7)
- moved D402 8.24 mm to (48.3, 17.0), turned to 0 degrees
Connections:
- removed net BATLVL: U401.15
- removed net CHARGE_STAT+: D301.A, R053.2
- removed net CHARGE_STAT-: D301.C, U301.1
- removed net EN: S201.5, U201.3
- removed net N$2: R301.2, U301.5
- removed net PWMB: R402.8, U401.31
- removed net PWMG: R402.5, U401.1
- removed net PWMR: R402.7, U401.38
- removed net VLIPO: C301.1, C449.2, D302.2, J301.2, U301.3, U401.49
- new net MCD: J401.4, U401.53
- new net PWMB/MC1: J401.1, R402.8, U401.31
- new net PWMG/MC2: J401.2, R402.5, U401.1
- new net PWMR/MC3: J401.3, R402.7, U401.38
- net BSL: now also J401.12; no longer J401.8
- net CONN_D+: now also R053.4; no longer R053.8
- net EXT: now also J401.15; no longer J401.11
- net GND: now also J401.6, R053.3; no longer C301.2, J301.1, J401.2, R053.6, R301.1, S201.4, S458.P$1, S458.P$3, U301.2
- net N$7: now also R053.2; no longer R053.3
- net RX0: now also J401.8; no longer J401.4
- net RX_GPS: now also J401.9; no longer J401.5
- net SCL0: now also J401.13; no longer J401.9
- net SDA0: now also J401.14; no longer J401.10
- net TX0: now also J401.7; no longer J401.3
- net TX_GPS: now also J401.10; no longer J401.6
- net USB_ON: no longer S458.P$2
- net VBUS: now also D402.1; no longer D302.1, D402.C, R053.7, U301.4
- net VCC: now also C449.2, J401.11, U401.49; no longer J401.7
- net VEXT: now also D402.2, J401.5; no longer D402.A, J401.1
- net VIN: now also D402.3, U201.3; no longer D302.3, S201.6
Routing:
- removed copper zone on layer 1, net GND
- removed copper zone on layer 16, net GND
Other:
- board text added: "Project Yukari"
- board text removed: "Charge"
- board text removed: "HighAcc"
- board text removed: "On"
- board text removed: "RocketometerMPU9150"

Commit message: More work on Yukari, replaced transistor with my own library, which includes SC70 package
Parts:
- Q050: device SparkFun:SOT23-3 -> KwanSystems:SC-70-3
- turned C201 to 0 degrees
- turned Q050 to 0 degrees
Connections:
- net N$6 renamed USB_CONNECT+
- net N$7 renamed USB_LED-
Routing:
- net VCC: track 0.00 -> 149.5 mm, vias 0 -> 14
- net SDA0: track 0.00 -> 89.7 mm, vias 0 -> 5
- net SCL0: track 0.00 -> 69.4 mm, vias 0 -> 4
- net PWMG/MC2: track 0.00 -> 65.3 mm, vias 0 -> 4
- net EXT: track 0.00 -> 48.6 mm, vias 0 -> 2
- net 1.8V: track 0.00 -> 46.3 mm, vias 0 -> 4
- net ONOFF: track 0.00 -> 41.6 mm, vias 0 -> 4
- net PPS: track 0.00 -> 30.9 mm, vias 0 -> 2
- net RX_GPS: track 0.00 -> 30.6 mm, vias 0 -> 2
- net TX_GPS: track 0.00 -> 29.7 mm, vias 0 -> 4
- net PWMB/MC1: track 0.00 -> 27.2 mm, vias 0 -> 3
- net PWMR/MC3: track 0.00 -> 26.2 mm, vias 0 -> 3
- net RESET: track 0.00 -> 23.7 mm, vias 0 -> 4
- net ACCINT: track 0.00 -> 22.7 mm
- net USB_SOFTCONNECT: track 0.00 -> 22.5 mm, vias 0 -> 1
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- added copper zone on layer 1, net GND
- added copper zone on layer 16, net GND
Other:
- board text added: "MC1"
- board text added: "MC2"
- board text added: "MC3"
- board text added: "MCD"

Commit message: Added new feature to NavCalc
Parts:
- removed C302: 4.7uF, SparkFun:0402-CAP
- removed C901: 10uF, SparkFun:0603-CAP
- removed C906: 100nF, SparkFun-Passives:0402-CAP
- removed R011: 100k, SparkFun:0402-RES
- removed U$5: (no value), KwanSystems:KWAN_ACC
- removed U$6: (no value), KwanSystems:OSHW_ACC
- removed U902: ADXL375, KwanSystems:ADXL375
- D402: value DIODE_COMMON_CATHODEBAT30C -> (none); device KwanSystems:SC-70-3 -> KwanSystems:D0603
- moved C505 30.5 mm to (10.9, 2.29), turned to 270 degrees
- moved C504 29.2 mm to (12.2, 2.29), turned to 90 degrees
- moved U501 26.8 mm to (14.7, 2.29), turned to 270 degrees
- moved C501 24.5 mm to (17.5, 2.29), turned to 270 degrees
- moved D402 13.6 mm to (34.8, 18.8)
- moved C101 12.8 mm to (20.8, 17.8), turned to 180 degrees
- moved U101 12.7 mm to (20.8, 15.0), turned to 270 degrees
Connections:
- removed net VIN: C201.1, D402.3, U201.1, U201.3
- net GND: no longer C302.2, C901.2, C906.2, R011.1, U902.12, U902.2, U902.4, U902.5
- net SCL0: no longer U902.14
- net SDA0: no longer U902.13
- net USB_ON: no longer R015.2
- net VBUS: now also C201.1, U201.1, U201.3; no longer C302.1, D402.1, R011.2, R015.3
- net VCC: no longer C901.1, C906.1, U902.1, U902.6, U902.7
- net VEXT: now also D402.A; no longer D402.2
Routing:
- net SDA0: track 89.7 -> 52.1 mm
- net 1.8V: track 46.3 -> 11.2 mm, vias 4 -> 2
- net PWMR/MC3: track 26.2 -> 58.1 mm
- net RX_GPS: track 30.6 -> 58.6 mm
- net MCD: track 20.4 -> 46.3 mm, vias 1 -> 4
- net SCL0: track 69.4 -> 44.9 mm, vias 4 -> 2
- net VIN: track 19.7 -> 0.00 mm, vias 2 -> 0
- net PPS: track 30.9 -> 50.0 mm
- net ONOFF: track 41.6 -> 57.8 mm, vias 4 -> 2
- net PWMG/MC2: track 65.3 -> 51.8 mm, vias 4 -> 5
- net USB_ON: track 13.2 -> 0.00 mm, vias 1 -> 0
- net ACCINT: track 22.7 -> 34.6 mm, vias 0 -> 2
- net SCK0: track 9.15 -> 20.9 mm
- net EXT: track 48.6 -> 37.6 mm, vias 2 -> 3
- net VEXT: track 13.1 -> 3.35 mm, vias 1 -> 0
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Other:
- board text added: "v1.0 10 Apr 2014"
- board text removed: "v1.0 01 Apr 2014"
