File: KwanSystems/Yukari/Yukari 3 11DoF.sch (EAGLE design)
At the start: 55 parts, among them J001 M06, J003 M06, J301 JST 2mm, J406 11DoF, J501 GP-2106, Q601 SSM6N58NU, U201 5319, U301 73831, U401 LPC2148, U501 5319 1.8V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

Commit message: More work to Yukari3
Parts:
- removed Q601: SSM6N58NU, KwanSystems:SSM6N58NU
- removed R601: 220, KwanSystems:RP2EXB24V
- removed R602: 10k, KwanSystems:RP404
- removed U601: OPTO, SparkFun:OPTOISOLATOR-2SOIC8
- added C1, C3: 100nF, SparkFun:CAP0402-CAP
- added C2: 10uF, SparkFun-Capacitors:10UF-6.3V-20%(1206)
- added J502: (no value), SparkFun-Connectors:M03PTH
- added U600: ADUM3221, KwanSystems:ADUM3221
- J001: device SparkFun:M06SIP -> SparkFun-Connectors:M18_
- R401: value 10k -> (none); device KwanSystems:RP404 -> KwanSystems:RP2EXB24V
- renumbered JP5 to J605, JP6 to J602, JP7 to J600
Connections:
- net AD1 renamed IC
- net AD2 renamed IG
- net AD3 renamed IA
- removed net N$11: R601A.2, U601.A1
- removed net N$13: R601B.2, U601.A2
- removed net OUT1: J602.1, Q601B.D, R602A.1
- removed net OUT1N: Q601B.G, R602C.1, U601.CL1
- removed net OUT2: J605.1, Q601A.D, R602B.1
- removed net OUT2N: Q601A.G, R602D.1, U601.CL2
- removed net SERVO1: R601A.1, U401.(SSEL0/PWM2/EINT2)P0.7
- removed net SERVO2: R601B.1, U401.(PWM5/AD1.6/CAP1.3)P0.21
- new net PWM2: U401.(SSEL0/PWM2/EINT2)P0.7, U600A.IN
- new net PWM5: U401.(PWM5/AD1.6/CAP1.3)P0.21, U600B.IN
- new net QWM2: J602.1, U600A.OUT
- new net QWM5: J605.1, U600B.OUT
- net BSL: no longer R401B.2
- net CS0: no longer U401.P0.23
- net GND: now also C1.2, J502.1, U600INP.GND; no longer U601.C1, U601.C2
- net HV: now also C2.1, C3.1, U600OUTP.VCC; no longer R602A.2, R602B.2, R602C.2, R602D.2
- net HV-GND: now also C2.2, C3.2, U600OUTP.GND; no longer Q601A.S, Q601B.S, U601.EM1, U601.EM2
- net RST: now also R401B.2; no longer R401D.2
- net RX1: now also J502.2
- net TX1: now also J502.3
- net VCC: now also C1.1, U600INP.VCC; no longer R401C.1, R401D.1
Other:
- moved on the sheet: R401A, R401B
