File: KwanSystems/Yukari/Tomo5.sch (EAGLE design)
At the start: 39 parts, among them J101 USB_MICROB_JST, U101 FT232RLSSOP, U401 ATMEGA328P, U501 FGPMMOPA6H, U601 MPU9250, X501 uFL, Y401 16MHz

Commit message: Added Adafruit stuff
Parts:
- removed LOGO1: SFE_LOGO_FLAME.1_INCH, SparkFun-Aesthetics:SFE_LOGO_FLAME.1_INCH
- removed LOGO2: OSHW-LOGOS, SparkFun-Aesthetics:OSHW-LOGOS
- removed R501: 680, SparkFun-Passives:RESISTOR0402-RES
- removed STANDOFF1, STANDOFF2: STAND-OFF, SparkFun-Electromechanical:STAND-OFF
- added D001: RED, SparkFun-LED:LED0603
- added D002: GREEN, SparkFun-LED:LED0603
- added D403: YELLOW, SparkFun-LED:LED0603
- added J002, J003: (no value), SparkFun-Connectors:M03PTH
- added R001: 680, KwanSystems:RP404
- added R002: 10k, SparkFun-Passives:RESISTOR0402-RES
- added U$7: ADUM3221, KwanSystems:ADUM3221
- C502: device microbuilder:CAP_CERAMIC0805-NOOUTLINE -> SparkFun-Capacitors:CAP1206
- renumbered U$12 to J001
Connections:
- net 3V3 renamed 3.3V
- net D0 renamed D0/AT_RX
- net D1 renamed D1/AT_TX
- net D13 renamed D13/ENC0_ECHO+
- net N$8 renamed ENC0_ECHO-
- net SCL renamed A5/SCL
- net SDA renamed A4/SDA
- removed net D2: U401.PD2(INT0)
- removed net D5: U401.PD5(T1)
- removed net D6: U401.PD6(AIN0)
- removed net ENC0: J400.2, U401.PC0(ADC0)
- removed net ENC1: J401.2, U401.PC3(ADC3)
- removed net N$11: D122.A, R101B.1
- removed net N$9: D123.A, R101A.1
- removed net RXLED1: R101B.2, U101.RXLED
- removed net TXLED1: R101A.2, U101.TXLED
- new net A0/ENC0: J400.1, U401.PC0(ADC0)
- new net A3/ENC1: J401.1, U401.PC3(ADC3)
- new net D2/ENC1_ECHO+: R001C.2, U401.PD2(INT0)
- new net D5/STEER+: U$7A.IN, U401.PD5(T1)
- new net D6/THROTTLE+: U$7B.IN, U401.PD6(AIN0)
- new net GND-ISO: J002.3, J003.3, R002.1, U$7OUTP.GND
- new net IPWR-: D002.C, R002.2
- new net N$8: D403.A, R001C.1
- new net PPS_ECHO-: D001.C, R001B.1
- new net RXLED+: D123.C, R101A.1
- new net RXLED-: R101A.2, U101.RXLED
- new net STEER-: J003.1, U$7A.OUT
- new net THROTTLE-: J002.1, U$7B.OUT
- new net TXLED+: D122.C, R101B.1
- new net TXLED-: R101B.2, U101.TXLED
- new net VCC-ISO: D002.A, J002.2, J003.2, U$7OUTP.VCC
- net 5V: now also D122.A, D123.A, D401.A, J400.2, J401.2, U$7INP.VCC; no longer D122.C, D123.C, J400.1, J401.1, R101C.2
- net GND: now also D403.C, R001A.2, R001B.2, R101C.2, U$7INP.GND; no longer D401.C, R501.1
- net N$5: now also D401.C; no longer D401.A
- net N$6: now also R001A.1; no longer R501.2
- net PPS_ECHO+: now also D001.A
Other:
- moved on the sheet: C502, D122, D123, D401, D402, L501, R101A, R101B, R101C, R101D
