File: KwanSystems/Yukari/Yukari4 Naninator.sch (EAGLE design)
At the start: 42 parts, among them J001 USB_MICROB_JST, J501 GP-2106, J502 UP501, U001 FT232RLSSOP, U002 100nF, U003 100nF, U101 MPU-9250, U401 ATMEGA328P, U501 ADUM242E, U502 V_REG_LDOSMD2, U516 100nF, U521 100nF, U601 ADUM3221, Y401 16MHz

Commit message: More progress
Parts:
- removed C511: 0.1uF, SparkFun:CAP0402-CAP
- removed C512, C552: 10uF, SparkFun:CAP_POL1206
- removed C551: 1uF, SparkFun:CAP0402-CAP
- removed U$1: THR_SERVO_CONN, KwanSystems:THR_SERVO_CONN
- removed U502: V_REG_LDOSMD2, SparkFun:V_REG_LDOSMD2
- added C211, C221: 1uF, SparkFun:CAP0402-CAP
- added C214, C224: 100nF, SparkFun:CAP0402-CAP
- added C215, C225, C303, C304: 4.7uF, SparkFun:CAP0402-CAP
- added D301: YELLOW, SparkFun:LED0603
- added D302: PMEG2005CT, KwanSystems:DIODE_COMMON_CATHODEPMEG2005CT
- added J002: USB_MICROB_JST, KwanSystems:USB_MICROB_JST
- added J301: JST 2mm, SparkFun:M02-JST-2MM-SMT
- added JP3: T, SparkFun-Connectors:M03PTH
- added R304: 1.5k, SparkFun:RESISTOR0402-RES
- added R305, R6: 10k, SparkFun:RESISTOR0402-RES
- added S2: B3U-1000P, KwanSystems:B3U-1000P
- added S201: AYZ0202, KwanSystems:AYZ0202
- added U201: 3.3V, KwanSystems:MIC5319D5
- added U202: 1.8V, KwanSystems:MIC5319D5
- added U301: MCP73831, KwanSystems:MCP73831
- C110, C113: device SparkFun-Capacitors:0.1UF-25V(+80/-20%)(0603) -> SparkFun-Capacitors:CAP0402-CAP
- JP5: value STEERING -> S
- renumbered U$3 to J101, U002 to C601, U003 to C608
Connections:
- removed net N$14: U501PWR1.GND, U521.1
- removed net N$15: U501PWR2.GND, U516.1
- new net BYP1.8: C224.1, U202.BYP
- new net BYP3.3: C214.1, U201.BYP
- new net GGND: C211.2, C214.2, C215.2, C221.2, C224.2, C225.2, C303.2, C304.2, J002.GND, J301.1, R305.1, S201A.P$1, S201B.P$2, U201.GND, U202.GND, U301.VSS, U501PWR1.GND, U521.1
- new net N$10: R305.2, U301.PROG
- new net N$12: D301.C, U301.STAT
- new net N$13: D301.A, R304.1
- new net PWR_EN1.8: S201B.P$3, U202.EN
- new net PWR_EN3.3: S201A.P$3, U201.EN
- new net VBUS: C304.1, D302.A1, J002.VBUS, R304.2, U301.VIN
- new net VGPS: C008.+, C215.1, C225.1, J502.BAT, J502.VDD, U201.VOUT, U202.VOUT, U501PWR1.VCC, U521.2
- new net VIN: C211.1, C221.1, D302.K, S201A.P$2, S201B.P$1, U201.VIN, U202.VIN
- new net VLIPO: C303.1, D302.A2, J301.2, U301.VBAT
- net 1.8V: no longer C551.1, C552.+, U501PWR1.VCC, U502.OUT, U521.2
- net 3.3V: now also R6.2; no longer C511.1, C512.+, J502.BAT, J502.VDD, U502.EN, U502.IN
- net GND: now also C008.-, S2.2, U501PWR2.GND, U516.1; no longer C511.2, C512.-, C551.2, C552.-, U502.GND
- net N$6: now also U601B.OUT; no longer U601A.OUT
- net N$7: now also JP3.3, U601A.OUT; no longer U$1.SIGNAL, U601B.OUT
- net ONOFF: now also R6.1, S2.1
- net PGND: now also JP3.1; no longer U$1.GND, U$1.NC
- net PVCC: now also JP3.2; no longer U$1.VCC
- net S_SERVO: now also U601B.IN; no longer U601A.IN
- net T_SERVO: now also U601A.IN; no longer U601B.IN
Other:
- note added: "For R301=10k, Ireg=1000V/10000Ohm=0.1A"
- note added: "Max charge current Ireg=1000V/R301"
- note added: "Section 0 - USB interface"
- note added: "Section 2 - Regulator"
- note added: "Section 3 - Charging circuit"
- note removed: "1.8V"
- moved on the sheet: C008

Commit message: Added Adafruit stuff
Parts:
- removed J002: USB_MICROB_JST, KwanSystems:USB_MICROB_JST
- removed S2: B3U-1000P, KwanSystems:B3U-1000P
- added J302: USB_MICROB_JST, KwanSystems:USB_MICROB_JST
- added S501: B3U-1000P, KwanSystems:B3U-1000P
- C110, C113: value 0.1uF -> 100nF
- U101: value MPU-9250 -> MPU9250; device Testing:MPU-9250 -> KwanSystems:MPU9250
Connections:
- net VIN renamed VIN_GPS
- removed net 1.8V: J501.VCC
- removed net AUX_CL: U101.AUX_CL
- removed net AUX_DA: U101.AUX_DA
- removed net FSYNC: U101.FSYNC
- new net TX_I: J502.TXD
- net 1PPS_I: now also J502.PPS
- net 3.3V: now also U101.#CS; no longer U101.!CS
- net GGND: now also J302.GND; no longer J002.GND
- net GND: now also S501.2; no longer S2.2
- net ONOFF: now also S501.1; no longer S2.1
- net PPS: no longer J502.PPS
- net RX_GPS: no longer J502.RXD
- net RX_I: now also J502.RXD
- net TX_GPS: no longer J502.TXD
- net VBUS: now also J302.VBUS; no longer J002.VBUS
- net VGPS: now also J501.VCC
Other:
- note added: "Controller side"
- note added: "GPS side"
- note removed: "High voltage (controller) side"
- note removed: "Low voltage (GPS) side"
- note removed: "Section 0 - USB interface"
- moved on the sheet: C008, C221, C224, C225, J501, J502, R6, S201B, U202, U516, U521
