File: KwanSystems/LPC2368 Breakout.brd (EAGLE design)
At the start: 71.1 x 30.5 mm, 69 parts, among them J001 USB_MICROB_JST, J301 JST 2mm, J401 M13, J402 M12PTH, J403 M13, J404 M12PTH, J405 M13, J406 M12PTH, J407 M13, J408 M12PTH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

Commit message: Reorganized docs for ARM. Added engine rooms with AD magnetic couplers instead of optocouplers.
Parts:
- removed Q201: PMOS, SparkFun:SOT23-3
- added C416, C418: 18pF, SparkFun-Passives:0402-CAP
- added C502: 4.7uF, SparkFun:0402-CAP
- added R417: 10k, SparkFun:0402-RES
- added U501: 1525, KwanSystems:SOT-23-3
- added Y416: 32kiHz, SparkFun:CRYSTAL-32KHZ-SMD
- R010: value 10k -> 24k
- R011: value 100k -> 39k
- turned Y422 to 90 degrees
Connections:
- removed net RAW: C201.1, Q201.3, U201.1, U201.3
- net ADREF: now also C502.1, U501.2
- net AGND: now also C502.2, U501.3
- net GND: now also C416.1, C418.1, S417.P$2
- net N$18: now also U201.3; no longer Q201.1
- net RESET: now also R417.2, S417.P$1
- net RTCX1: now also C416.2, Y416.X1
- net RTCX2: now also C418.2, Y416.X2
- net USB_ON: now also R011.2
- net VBUS: no longer R011.2
- net VDD(DCDC): now also R417.1
- net VDDA: now also U501.1
- net VIN-: now also C201.1, U201.1; no longer Q201.2
- net XTAL1: now also Y422.1; no longer Y422.3
- net XTAL2: now also Y422.3; no longer Y422.1
Routing:
- net RESET: track 17.8 -> 37.9 mm, vias 1 -> 2
- net RAW: track 9.39 -> 0.00 mm
- net RTCX1: track 14.7 -> 21.7 mm
- net RTCX2: track 14.5 -> 21.0 mm
- net VIN-: track 12.5 -> 18.2 mm
- net ADREF: track 4.26 -> 7.33 mm
- net VDDA: track 39.7 -> 40.8 mm
- net N$18: track 3.08 -> 2.27 mm
- net VBUS: track 22.0 -> 21.3 mm

Commit message: Fixed switch direction
Parts:
- added S001: SOLDERJUMPERNO, SparkFun-Passives:SJ_2S-NO
- S201: value SPDT -> AYZ0202; device SparkFun:AYZ0202 -> KwanSystems:AYZ0202
- Y416: device SparkFun:CRYSTAL-32KHZ-SMD -> KwanSystems:ABS06
- moved C416 0.80 mm to (26.7, 10.7)
- moved C418 0.80 mm to (26.7, 7.11)
- turned C201 to 0 degrees
Connections:
- net GND: now also S001.1, S201.1; no longer S201.3
- net RTCX1: now also S001.2, Y416.1; no longer Y416.X1
- net RTCX2: now also Y416.2; no longer Y416.X2
- net VIN-: now also S201.3; no longer S201.1
Routing:
- net N$18: track 2.27 -> 7.94 mm
- net VIN-: track 18.2 -> 21.6 mm
- net RTCX1: track 21.7 -> 23.8 mm
- net USB_CONNECT: track 40.9 -> 42.2 mm
- net USB_ON: track 61.8 -> 63.1 mm
- net RTCX2: track 21.0 -> 20.3 mm
Other:
- board text added: "12 Jul 2014"
- board text added: "LPC2368 Breakout v2"
- board text removed: "13 Apr 2012"
- board text removed: "LPC2368 Breakout"
