File: KwanSystems/LQFP100 Breakout.sch (EAGLE design)
At the start: 9 parts, among them U1 LPC2368

Commit message: Added LegoClassicSpace.svg after checking local copy. We'll see how the pull works
Connections:
- net N$100: now also U1.RTCK; no longer U1.P1[9]/ENET_RXD0
- net N$73: now also U1.P2[2]/PWM1[3]/CTS1/PIPESTAT1; no longer U1.RTCK
- net N$74: now also U1.P2[1]/PWM1[2]/RXD1/PIPESTAT0; no longer U1.P0[3]/RXD0
- net N$75: now also U1.P2[0]/PWM1[1]/TXD1/TRACECLK; no longer U1.P0[2]/TXD0
- net N$76: now also U1.P0[9]/I2STX_SDA/MOSI1/MAT2[3]; no longer U1.GND6
- net N$77: now also U1.P0[8]/I2STX_WS/MISO1/MAT2[2]; no longer U1.VDD(3V3)3
- net N$78: now also U1.P0[7]/I2STX_CLK/SCK1/MAT2[1]; no longer U1.P1[0]/ENET_TXD0
- net N$79: now also U1.P0[6]/I2SRX_SDA/SSEL1/MAT2[0]; no longer U1.P1[1]/ENET_TXD1
- net N$80: now also U1.P0[5]/I2SRX_WS/TD2/CAP2[1]; no longer U1.P1[4]/ENET_TX_EN
- net N$81: now also U1.P0[4]/I2SRX_CLK/RD2/CAP2[0]; no longer U1.P1[8]/ENET_CRS
- net N$82: now also U1.P4[28]/MAT2[0]/TXD3; no longer U1.P2[2]/PWM1[3]/CTS1/PIPESTAT1
- net N$83: now also U1.GND6; no longer U1.P2[1]/PWM1[2]/RXD1/PIPESTAT0
- net N$84: now also U1.VDD(DCDC)2; no longer U1.P2[0]/PWM1[1]/TXD1/TRACECLK
- net N$85: now also U1.P4[29]/MAT2[1]/RXD3; no longer U1.P0[9]/I2STX_SDA/MOSI1/MAT2[3]
- net N$86: now also U1.P1[17]/ENET_MDIO; no longer U1.P0[8]/I2STX_WS/MISO1/MAT2[2]
- net N$87: now also U1.P1[16]/ENET_MDC; no longer U1.P0[7]/I2STX_CLK/SCK1/MAT2[1]
- net N$88: now also U1.P1[15]/ENET_REF_CLK; no longer U1.P0[6]/I2SRX_SDA/SSEL1/MAT2[0]
- net N$89: now also U1.P1[14]/ENET_RX_ER; no longer U1.P0[5]/I2SRX_WS/TD2/CAP2[1]
- net N$90: now also U1.P1[10]/ENET_RXD1; no longer U1.P0[4]/I2SRX_CLK/RD2/CAP2[0]
- net N$91: now also U1.P1[9]/ENET_RXD0; no longer U1.P4[28]/MAT2[0]/TXD3
- net N$92: now also U1.P1[8]/ENET_CRS; no longer U1.GND5
- net N$93: now also U1.P1[4]/ENET_TX_EN; no longer U1.VDD(DCDC)2
- net N$94: now also U1.P1[1]/ENET_TXD1; no longer U1.P4[29]/MAT2[1]/RXD3
- net N$95: now also U1.P1[0]/ENET_TXD0; no longer U1.P1[17]/ENET_MDIO
- net N$96: now also U1.VDD(3V3)3; no longer U1.P1[16]/ENET_MDC
- net N$97: now also U1.GND5; no longer U1.P1[15]/ENET_REF_CLK
- net N$98: now also U1.P0[2]/TXD0; no longer U1.P1[14]/ENET_RX_ER
- net N$99: now also U1.P0[3]/RXD0; no longer U1.P1[10]/ENET_RXD1
